File: PC_ExtensionBoard/PC_ExtensionBoard.kicad_pcb (KiCad board)
At the start: 2 copper layers, 128.2 x 98.2 mm, 10 parts, among them U1 HC-USB3.0-L168-WP, U2 10GHz, U3 KBLH-E61_COMe_Type6_16U

Commit message: update Schematic
Parts:
- USB1: footprint ACLAB:USB-A-TH_H181-AF2R06-12ALCR -> PC_ExtensionBoard:USB-A-TH_H181-AF2R06-12ALCR
Connections:
- U1 pad 1: unconnected-(U1-VBUS-Pad1) -> /USB_Audio_RJ45/P2_VBUS
- U1 pad 10: unconnected-(U1-SH-Pad10) -> GND
- U1 pad 2: unconnected-(U1-D--Pad2) -> /USB_Audio_RJ45/P2_D-
- U1 pad 3: unconnected-(U1-D+-Pad3) -> /USB_Audio_RJ45/P2_D+
- U1 pad 4: unconnected-(U1-GND-Pad4) -> GND
- U1 pad 5: unconnected-(U1-SSRX--Pad5) -> /PC_CoreBoard/USBSS2.RX-
- U1 pad 6: unconnected-(U1-SSRX+-Pad6) -> /PC_CoreBoard/USBSS2.RX+
- U1 pad 7: unconnected-(U1-GND_DRAN-Pad7) -> GND
- U1 pad 8: unconnected-(U1-SSTX--Pad8) -> /PC_CoreBoard/USBSS2.TX-
- U1 pad 9: unconnected-(U1-SSTX+-Pad9) -> /PC_CoreBoard/USBSS2.TX+
- U3 pad A1: unconnected-(U3A-GND-PadA1) -> GND
- U3 pad A10: unconnected-(U3G-GBE0_MDI1+-PadA10) -> /PC_CoreBoard/GBE0.MDI1+
- U3 pad A104: unconnected-(U3A-VCC_12V-PadA104) -> /PC_CoreBoard/VCC_12V
- U3 pad A105: unconnected-(U3A-VCC_12V-PadA105) -> /PC_CoreBoard/VCC_12V
- U3 pad A106: unconnected-(U3A-VCC_12V-PadA106) -> /PC_CoreBoard/VCC_12V
- U3 pad A107: unconnected-(U3A-VCC_12V-PadA107) -> /PC_CoreBoard/VCC_12V
- U3 pad A108: unconnected-(U3A-VCC_12V-PadA108) -> /PC_CoreBoard/VCC_12V
- U3 pad A109: unconnected-(U3A-VCC_12V-PadA109) -> /PC_CoreBoard/VCC_12V
- U3 pad A11: unconnected-(U3A-GND-PadA11) -> GND
- U3 pad A110: unconnected-(U3A-GND-PadA110) -> GND
- U3 pad A12: unconnected-(U3G-GBE0_MDI0--PadA12) -> /PC_CoreBoard/GBE0.MDI0-
- U3 pad A13: unconnected-(U3G-GBE0_MDI0+-PadA13) -> /PC_CoreBoard/GBE0.MDI0+
- U3 pad A14: unconnected-(U3G-GBE0_CTREF-PadA14) -> /PC_CoreBoard/GBE0.CTREF
- U3 pad A2: unconnected-(U3G-GBE0_MDI3--PadA2) -> /PC_CoreBoard/GBE0.MDI3-
- U3 pad A21: unconnected-(U3A-GND-PadA21) -> GND
- U3 pad A3: unconnected-(U3G-GBE0_MDI3+-PadA3) -> /PC_CoreBoard/GBE0.MDI3+
- U3 pad A31: unconnected-(U3A-GND-PadA31) -> GND
- U3 pad A38: unconnected-(U3C-USB_6_7_OC#-PadA38) -> /PC_CoreBoard/USB_6_7_OC#
- U3 pad A41: unconnected-(U3A-GND-PadA41) -> GND
- U3 pad A44: unconnected-(U3C-USB_2_3_OC#-PadA44) -> /PC_CoreBoard/USB_2_3_OC#
- U3 pad A5: unconnected-(U3G-GBE0_LINK1000#-PadA5) -> /PC_CoreBoard/~{GBE0_LINK_1000}
- U3 pad A51: unconnected-(U3A-GND-PadA51) -> GND
- U3 pad A52: unconnected-(U3I-PCIE_TX5+-PadA52) -> /PC_CoreBoard/PCIe_{B1x2}.RX1+
- U3 pad A53: unconnected-(U3I-PCIE_TX5--PadA53) -> /PC_CoreBoard/PCIe_{B1x2}.RX1-
- U3 pad A55: unconnected-(U3I-PCIE_TX4+-PadA55) -> /PC_CoreBoard/PCIe_{B1x2}.RX0+
- U3 pad A56: unconnected-(U3I-PCIE_TX4--PadA56) -> /PC_CoreBoard/PCIe_{B1x2}.RX0-
- U3 pad A57: unconnected-(U3A-GND-PadA57) -> GND
- U3 pad A58: unconnected-(U3I-PCIE_TX3+-PadA58) -> /PC_CoreBoard/PCIe_{B1x4}.RX3+
- U3 pad A59: unconnected-(U3I-PCIE_TX3--PadA59) -> /PC_CoreBoard/PCIe_{B1x4}.RX3-
- U3 pad A6: unconnected-(U3G-GBE0_MDI2--PadA6) -> /PC_CoreBoard/GBE0.MDI2-
- U3 pad A60: unconnected-(U3A-GND-PadA60) -> GND
- U3 pad A61: unconnected-(U3I-PCIE_TX2+-PadA61) -> /PC_CoreBoard/PCIe_{B1x4}.RX2+
- U3 pad A62: unconnected-(U3I-PCIE_TX2--PadA62) -> /PC_CoreBoard/PCIe_{B1x4}.RX2-
- U3 pad A64: unconnected-(U3I-PCIE_TX1+-PadA64) -> /PC_CoreBoard/PCIe_{B1x4}.RX1+
- U3 pad A65: unconnected-(U3I-PCIE_TX1--PadA65) -> /PC_CoreBoard/PCIe_{B1x4}.RX1-
- U3 pad A66: unconnected-(U3A-GND-PadA66) -> GND
- U3 pad A68: unconnected-(U3I-PCIE_TX0+-PadA68) -> /PC_CoreBoard/PCIe_{B1x4}.RX0+
- U3 pad A69: unconnected-(U3I-PCIE_TX0--PadA69) -> /PC_CoreBoard/PCIe_{B1x4}.RX0-
- U3 pad A7: unconnected-(U3G-GBE0_MDI2+-PadA7) -> /PC_CoreBoard/GBE0.MDI2+
- U3 pad A70: unconnected-(U3A-GND-PadA70) -> GND
- U3 pad A8: unconnected-(U3G-GBE0_LINK#-PadA8) -> /PC_CoreBoard/~{GBE0_LINK}
- U3 pad A80: unconnected-(U3A-GND-PadA80) -> GND
- U3 pad A9: unconnected-(U3G-GBE0_MDI1--PadA9) -> /PC_CoreBoard/GBE0.MDI1-
- U3 pad A90: unconnected-(U3A-GND-PadA90) -> GND
- U3 pad B1: unconnected-(U3A-GND-PadB1) -> GND
- U3 pad B104: unconnected-(U3A-VCC_12V-PadB104) -> /PC_CoreBoard/VCC_12V
- U3 pad B105: unconnected-(U3A-VCC_12V-PadB105) -> /PC_CoreBoard/VCC_12V
- U3 pad B106: unconnected-(U3A-VCC_12V-PadB106) -> /PC_CoreBoard/VCC_12V
- U3 pad B107: unconnected-(U3A-VCC_12V-PadB107) -> /PC_CoreBoard/VCC_12V
- U3 pad B108: unconnected-(U3A-VCC_12V-PadB108) -> /PC_CoreBoard/VCC_12V
- U3 pad B109: unconnected-(U3A-VCC_12V-PadB109) -> /PC_CoreBoard/VCC_12V
- U3 pad B11: unconnected-(U3A-GND-PadB11) -> GND
- U3 pad B110: unconnected-(U3A-GND-PadB110) -> GND
- U3 pad B2: unconnected-(U3G-GBE0_ACT#-PadB2) -> /PC_CoreBoard/~{GBE0_ACT}
- U3 pad B21: unconnected-(U3A-GND-PadB21) -> GND
- U3 pad B31: unconnected-(U3A-GND-PadB31) -> GND
- U3 pad B38: unconnected-(U3C-USB_4_5_OC#-PadB38) -> /PC_CoreBoard/USB_4_5_OC#
- U3 pad B41: unconnected-(U3A-GND-PadB41) -> GND
- U3 pad B44: unconnected-(U3C-USB_0_1_OC#-PadB44) -> /PC_CoreBoard/USB_0_1_OC#
- U3 pad B51: unconnected-(U3A-GND-PadB51) -> GND
- U3 pad B52: unconnected-(U3I-PCIE_RX5+-PadB52) -> /PC_CoreBoard/PCIe_{B1x2}.TX1+
- U3 pad B53: unconnected-(U3I-PCIE_RX5--PadB53) -> /PC_CoreBoard/PCIe_{B1x2}.TX1-
- U3 pad B55: unconnected-(U3I-PCIE_RX4+-PadB55) -> /PC_CoreBoard/PCIe_{B1x2}.TX0+
- U3 pad B56: unconnected-(U3I-PCIE_RX4--PadB56) -> /PC_CoreBoard/PCIe_{B1x2}.TX0-
- U3 pad B58: unconnected-(U3I-PCIE_RX3+-PadB58) -> /PC_CoreBoard/PCIe_{B1x4}.TX3+
- U3 pad B59: unconnected-(U3I-PCIE_RX3--PadB59) -> /PC_CoreBoard/PCIe_{B1x4}.TX3-
- U3 pad B60: unconnected-(U3A-GND-PadB60) -> GND
- U3 pad B61: unconnected-(U3I-PCIE_RX2+-PadB61) -> /PC_CoreBoard/PCIe_{B1x4}.TX2+
- U3 pad B62: unconnected-(U3I-PCIE_RX2--PadB62) -> /PC_CoreBoard/PCIe_{B1x4}.TX2-
- U3 pad B64: unconnected-(U3I-PCIE_RX1+-PadB64) -> /PC_CoreBoard/PCIe_{B1x4}.TX1+
- U3 pad B65: unconnected-(U3I-PCIE_RX1--PadB65) -> /PC_CoreBoard/PCIe_{B1x4}.TX1-
- U3 pad B68: unconnected-(U3I-PCIE_RX0+-PadB68) -> /PC_CoreBoard/PCIe_{B1x4}.TX0+
- U3 pad B69: unconnected-(U3I-PCIE_RX0--PadB69) -> /PC_CoreBoard/PCIe_{B1x4}.TX0-
- U3 pad B70: unconnected-(U3A-GND-PadB70) -> GND
- U3 pad B80: unconnected-(U3A-GND-PadB80) -> GND
- U3 pad B84: unconnected-(U3A-VCC_5V_SBY-PadB84) -> Net-(U3A-VCC_5V_SBY-PadB84)
- U3 pad B85: unconnected-(U3A-VCC_5V_SBY-PadB85) -> Net-(U3A-VCC_5V_SBY-PadB84)
- U3 pad B86: unconnected-(U3A-VCC_5V_SBY-PadB86) -> Net-(U3A-VCC_5V_SBY-PadB84)
- U3 pad B87: unconnected-(U3A-VCC_5V_SBY-PadB87) -> Net-(U3A-VCC_5V_SBY-PadB84)
- U3 pad B90: unconnected-(U3A-GND-PadB90) -> GND
- U3 pad C1: unconnected-(U3A-GND-PadC1) -> GND
- U3 pad C100: unconnected-(U3A-GND-PadC100) -> GND
- U3 pad C103: unconnected-(U3A-GND-PadC103) -> GND
- U3 pad C104: unconnected-(U3A-VCC_12V-PadC104) -> /PC_CoreBoard/VCC_12V
- U3 pad C105: unconnected-(U3A-VCC_12V-PadC105) -> /PC_CoreBoard/VCC_12V
- U3 pad C106: unconnected-(U3A-VCC_12V-PadC106) -> /PC_CoreBoard/VCC_12V
- U3 pad C107: unconnected-(U3A-VCC_12V-PadC107) -> /PC_CoreBoard/VCC_12V
- U3 pad C108: unconnected-(U3A-VCC_12V-PadC108) -> /PC_CoreBoard/VCC_12V
- U3 pad C109: unconnected-(U3A-VCC_12V-PadC109) -> /PC_CoreBoard/VCC_12V
- U3 pad C11: unconnected-(U3A-GND-PadC11) -> GND
- U3 pad C110: unconnected-(U3A-GND-PadC110) -> GND
- U3 pad C14: unconnected-(U3A-GND-PadC14) -> GND
- U3 pad C2: unconnected-(U3A-GND-PadC2) -> GND
- U3 pad C21: unconnected-(U3A-GND-PadC21) -> GND
- U3 pad C31: unconnected-(U3A-GND-PadC31) -> GND
- U3 pad C41: unconnected-(U3A-GND-PadC41) -> GND
- U3 pad C5: unconnected-(U3A-GND-PadC5) -> GND
- U3 pad C51: unconnected-(U3A-GND-PadC51) -> GND
- U3 pad C6: GND -> /PC_CoreBoard/USBSS1.RX-
- U3 pad C60: unconnected-(U3A-GND-PadC60) -> GND
- U3 pad C67: unconnected-(U3A-GND-PadC67) -> GND
- U3 pad C7: GND -> /PC_CoreBoard/USBSS1.RX+
- U3 pad C70: unconnected-(U3A-GND-PadC70) -> GND
- U3 pad C73: unconnected-(U3A-GND-PadC73) -> GND
- U3 pad C76: unconnected-(U3A-GND-PadC76) -> GND
- U3 pad C8: unconnected-(U3A-GND-PadC8) -> GND
- U3 pad C84: unconnected-(U3A-GND-PadC84) -> GND
- U3 pad C87: unconnected-(U3A-GND-PadC87) -> GND
- U3 pad C90: unconnected-(U3A-GND-PadC90) -> GND
- U3 pad C93: unconnected-(U3A-GND-PadC93) -> GND
- U3 pad C96: unconnected-(U3A-GND-PadC96) -> GND
- U3 pad D1: unconnected-(U3A-GND-PadD1) -> GND
- U3 pad D100: unconnected-(U3A-GND-PadD100) -> GND
- U3 pad D103: unconnected-(U3A-GND-PadD103) -> GND
- U3 pad D104: unconnected-(U3A-VCC_12V-PadD104) -> /PC_CoreBoard/VCC_12V
- U3 pad D105: unconnected-(U3A-VCC_12V-PadD105) -> /PC_CoreBoard/VCC_12V
- U3 pad D106: unconnected-(U3A-VCC_12V-PadD106) -> /PC_CoreBoard/VCC_12V
- U3 pad D107: unconnected-(U3A-VCC_12V-PadD107) -> /PC_CoreBoard/VCC_12V
- U3 pad D108: unconnected-(U3A-VCC_12V-PadD108) -> /PC_CoreBoard/VCC_12V
- U3 pad D109: unconnected-(U3A-VCC_12V-PadD109) -> /PC_CoreBoard/VCC_12V
- U3 pad D11: unconnected-(U3A-GND-PadD11) -> GND
- U3 pad D110: unconnected-(U3A-GND-PadD110) -> GND
- U3 pad D14: unconnected-(U3A-GND-PadD14) -> GND
- U3 pad D2: unconnected-(U3A-GND-PadD2) -> GND
- U3 pad D21: unconnected-(U3A-GND-PadD21) -> GND
- U3 pad D31: unconnected-(U3A-GND-PadD31) -> GND
- U3 pad D41: unconnected-(U3A-GND-PadD41) -> GND
- U3 pad D5: unconnected-(U3A-GND-PadD5) -> GND
- U3 pad D51: unconnected-(U3A-GND-PadD51) -> GND
- U3 pad D6: GND -> /PC_CoreBoard/USBSS1.TX-
- U3 pad D60: unconnected-(U3A-GND-PadD60) -> GND
- U3 pad D67: unconnected-(U3A-GND-PadD67) -> GND
- U3 pad D7: GND -> /PC_CoreBoard/USBSS1.TX+
- U3 pad D70: unconnected-(U3A-GND-PadD70) -> GND
- U3 pad D73: unconnected-(U3A-GND-PadD73) -> GND
- U3 pad D76: unconnected-(U3A-GND-PadD76) -> GND
- U3 pad D8: unconnected-(U3A-GND-PadD8) -> GND
- U3 pad D80: unconnected-(U3A-GND-PadD80) -> GND
- U3 pad D84: unconnected-(U3A-GND-PadD84) -> GND
- U3 pad D87: unconnected-(U3A-GND-PadD87) -> GND
- U3 pad D90: unconnected-(U3A-GND-PadD90) -> GND
- U3 pad D93: unconnected-(U3A-GND-PadD93) -> GND
- U3 pad D96: unconnected-(U3A-GND-PadD96) -> GND
- USB1 pad 1: GND -> /USB_Audio_RJ45/P1_VBUS
- USB1 pad 10: /PC_CoreBoard/USBSS0.TX+ -> /USB_Audio_RJ45/P0_VBUS
- USB1 pad 11: /PC_CoreBoard/USBSS0.TX- -> /USB_Audio_RJ45/P0_D-
- USB1 pad 12: unconnected-(USB1B-D+-Pad12) -> /USB_Audio_RJ45/P0_D+
- USB1 pad 13: /PC_CoreBoard/USBSS0.RX+ -> GND
- USB1 pad 15: GND -> /PC_CoreBoard/USBSS0.RX+
- USB1 pad 16: /USB_Audio/P0_D- -> GND
- USB1 pad 17: /USB_Audio/P0_D+ -> /PC_CoreBoard/USBSS0.TX-
- USB1 pad 18: /USB_Audio/P0_VBUS -> /PC_CoreBoard/USBSS0.TX+
- USB1 pad 19: unconnected-(USB1A-GND-Pad19) -> GND
- USB1 pad 2: GND -> /USB_Audio_RJ45/P1_D-
- USB1 pad 20: unconnected-(USB1B-GND-Pad20) -> GND
- USB1 pad 3: GND -> /USB_Audio_RJ45/P1_D+
- USB1 pad 5: GND -> /PC_CoreBoard/USBSS1.RX-
- USB1 pad 6: GND -> /PC_CoreBoard/USBSS1.RX+
- USB1 pad 7: /USB_Audio/P1_D- -> GND
- USB1 pad 8: /USB_Audio/P1_D+ -> /PC_CoreBoard/USBSS1.TX-
- USB1 pad 9: /USB_Audio/P1_VBUS -> /PC_CoreBoard/USBSS1.TX+
Other:
- copper layers 2 -> 8

Commit message: components placement R1
Parts:
- added A1: Mech_M2_2280_H2.5mm, PC_Components_1:Mech_M2_2280_H2.5mm, B.Cu at (143.0, 109.0)
- added A4: Mech_M2_2230_H2.5mm, PC_Components_1:Mech_M2_2230_H2.5mm, B.Cu at (93.4, 83.0)
- added C10: C_Pol_100u_10V_KEMET-T520-B, PC_Components_1:C_Pol_EIA-B, F.Cu at (88.0, 71.6)
- added C204: C_100n_0402, antmicro-footprints:C_0402_1005Metric, F.Cu at (151.4, 75.7)
- added C205: C_100n_0402, antmicro-footprints:C_0402_1005Metric, F.Cu at (160.0, 92.0)
- added C39: C_Pol_68u_16V_Panasonic-TQC-D, antmicro-footprints:C_Pol_EIA-D, F.Cu at (166.3, 75.3)
- added C40: C_22u_16V_0603, antmicro-footprints:C_0603_1608Metric, F.Cu at (163.2, 75.2)
- added C45: C_1u_0402, antmicro-footprints:C_0402_1005Metric, B.Cu at (160.2, 78.2)
- added C48: C_100n_0402, antmicro-footprints:C_0402_1005Metric, F.Cu at (163.1, 78.2)
- added C50: C_1u_0402, antmicro-footprints:C_0402_1005Metric, F.Cu at (157.6, 75.0)
- added C52: C_Pol_100u_10V_KEMET-T520-B, antmicro-footprints:C_Pol_EIA-B, F.Cu at (157.8, 72.7)
- added C57: C_1u_0402, antmicro-footprints:C_0402_1005Metric, F.Cu at (149.5, 74.8)
- added C58: C_22u_16V_0603, antmicro-footprints:C_0603_1608Metric, F.Cu at (173.1, 97.1)
- added C59: C_22u_16V_0603, antmicro-footprints:C_0603_1608Metric, F.Cu at (171.8, 97.1)
- added C61: 1uF/16V, PC_Components_1:C_0402_1005Metric, B.Cu at (156.4, 61.9)
- added C62: C_1u_0402, antmicro-footprints:C_0402_1005Metric, F.Cu at (167.8, 96.3)
- added C64: C_Pol_100u_10V_KEMET-T520-B, antmicro-footprints:C_Pol_EIA-B, F.Cu at (166.3, 98.7)
- added C66: C_1u_0402, antmicro-footprints:C_0402_1005Metric, F.Cu at (161.3, 124.7)
- added C67: C_1u_0402, antmicro-footprints:C_0402_1005Metric, F.Cu at (158.0, 97.2)
- added C69: C_1u_0402, antmicro-footprints:C_0402_1005Metric, F.Cu at (158.0, 128.1)
- added C7: C_Pol_100u_10V_KEMET-T520-B, PC_Components_1:C_Pol_EIA-B, F.Cu at (71.0, 71.6)
- added C70: C_1u_0402, antmicro-footprints:C_0402_1005Metric, F.Cu at (149.2, 103.8)
- added D10: 0402ESDA-05N, PC_Components_1:C_0402_1005Metric, B.Cu at (151.5, 68.5)
- added D11: 0402ESDA-05N, PC_Components_1:C_0402_1005Metric, B.Cu at (157.5, 68.5)
- added D12: PESD24VS1UL-N, PC_Components_1:C_0402_1005Metric, B.Cu at (150.4, 61.9)
- added D14: 0402ESDA-05N, PC_Components_1:C_0402_1005Metric, B.Cu at (153.5, 68.5)
- added D19: 0402ESDA-05N, PC_Components_1:C_0402_1005Metric, B.Cu at (155.5, 68.5)
- added D27: TPD2E2U06_SC70, PC_Components_1:SC70-3, F.Cu at (76.4, 72.0)
- added D28: TPD2E2U06_SC70, PC_Components_1:SC70-3, F.Cu at (82.4, 71.9)
- added D36: BAT54C, antmicro-footprints:SOT-23-3, B.Cu at (155.5, 73.8)
- added H1: Spacer_Drill3.7mm_H2.5mm_9774025151R, PC_Components_1:Spacer_Drill3.7mm_H2.5mm_9774025151R, B.Cu at (143.0, 109.0)
- added H10: Spacer_Drill3.7mm_H2.5mm_9774025151R, PC_Components_1:Spacer_Drill3.7mm_H2.5mm_9774025151R, F.Cu at (54.0, 141.0)
- added H11: Spacer_Drill3.7mm_H2.5mm_9774025151R, PC_Components_1:Spacer_Drill3.7mm_H2.5mm_9774025151R, F.Cu at (171.0, 141.0)
- added H12: Spacer_Drill3.7mm_H2.5mm_9774025151R, PC_Components_1:Spacer_Drill3.7mm_H2.5mm_9774025151R, F.Cu at (54.0, 54.0)
- added H13: Spacer_Drill3.7mm_H2.5mm_9774025151R, PC_Components_1:Spacer_Drill3.7mm_H2.5mm_9774025151R, F.Cu at (171.0, 116.0)
- added H3: Spacer_Drill3.7mm_H2.5mm_9774025151R, PC_Components_1:Spacer_Drill3.7mm_H2.5mm_9774025151R, B.Cu at (93.4, 83.0)
- added H6: Spacer_Drill3.7mm_H2.5mm_9774025151R, PC_Components_1:Spacer_Drill3.7mm_H2.5mm_9774025151R, F.Cu at (54.0, 75.5)
- added H7: Spacer_Drill3.7mm_H2.5mm_9774025151R, PC_Components_1:Spacer_Drill3.7mm_H2.5mm_9774025151R, F.Cu at (171.0, 54.0)
- added H8: Spacer_Drill3.7mm_H2.5mm_9774025151R, PC_Components_1:Spacer_Drill3.7mm_H2.5mm_9774025151R, F.Cu at (54.0, 116.0)
- added H9: Spacer_Drill3.7mm_H2.5mm_9774025151R, PC_Components_1:Spacer_Drill3.7mm_H2.5mm_9774025151R, F.Cu at (171.0, 75.5)
- added J100: Bus_M.2_2199230-2, PC_Components_1:Bus_M.2_Socket_Key_E_TE_2199230-6, B.Cu at (63.6, 83.0)
- added J2: Conn_01x04_Pin, Connector_Hirose:Hirose_DF13-04P-1.25DSA_1x04_P1.25mm_Vertical, F.Cu at (174.0, 122.2)
- added J8: Bus_M.2_1-2199230-6, PC_Components_1:Bus_M.2_Socket_Key_M_TE_1-2199230-6, B.Cu at (63.3, 109.0)
- added L2: L_1u8_14A_Coilcraft-XAL6030, antmicro-footprints:L_Coilcraft-XAL6030, F.Cu at (160.0, 83.0)
- added L3: L_1u8_6.8A_WE-MAPI-4020, antmicro-footprints:L_WE-MAPI-4020, F.Cu at (168.7, 93.4)
- added Q3: BSS138-7-F, antmicro-footprints:SOT-23-3, F.Cu at (146.9, 101.3)
- added Q4: SI7613DN-T1-GE3, antmicro-footprints:Vishay_PowerPAK_1212-8_Single, F.Cu at (150.6, 101.0)
- added R100: R_15k_0402, antmicro-footprints:R_0402_1005Metric, F.Cu at (158.1, 76.4)
- added R104: R_0R001_0805, antmicro-footprints:R_0805_2012Metric, F.Cu at (153.2, 72.7)
- added R107: R_15k_0402, antmicro-footprints:R_0402_1005Metric, F.Cu at (170.3, 99.4)
- added R108: R_10k_0402, antmicro-footprints:R_0402_1005Metric, F.Cu at (169.3, 99.4)
- added R109: R_110k_0402, antmicro-footprints:R_0402_1005Metric, F.Cu at (171.3, 99.4)
- added R110: R_15k_0402, antmicro-footprints:R_0402_1005Metric, F.Cu at (172.3, 99.4)
- added R113: R_0R001_0805, antmicro-footprints:R_0805_2012Metric, F.Cu at (161.7, 98.7)
- added R115: R_0R_0402, antmicro-footprints:R_0402_1005Metric, F.Cu at (147.3, 104.8)
- added R116: R_10k_0402, antmicro-footprints:R_0402_1005Metric, F.Cu at (145.4, 103.8)
- added R117: R_30k_0402, antmicro-footprints:R_0402_1005Metric, F.Cu at (147.3, 103.8)
- added R118: R_100k_0402, antmicro-footprints:R_0402_1005Metric, F.Cu at (150.0, 98.1)
- added R119: R_0R_0402, antmicro-footprints:R_0402_1005Metric, F.Cu at (158.0, 126.2)
- added R37: 10K/1%, PC_Components_1:R_0402_1005Metric, B.Cu at (154.4, 61.9)
- added R40: 1K/1%, PC_Components_1:R_0402_1005Metric, B.Cu at (158.5, 61.9)
- added R47: 24K/1%, PC_Components_1:C_0402_1005Metric, B.Cu at (152.4, 61.9)
- added R86: R_10k_0402, antmicro-footprints:R_0402_1005Metric, B.Cu at (158.8, 73.8)
- added R87: R_30k_0402, antmicro-footprints:R_0402_1005Metric, B.Cu at (157.8, 73.8)
- added R91: R_68k_0402, antmicro-footprints:R_0402_1005Metric, B.Cu at (158.8, 78.2)
- added R92: R_10k_0402, antmicro-footprints:R_0402_1005Metric, B.Cu at (157.8, 78.2)
- added R96: R_10k_0402, antmicro-footprints:R_0402_1005Metric, B.Cu at (162.0, 78.2)
- added R99: R_68k_0402, antmicro-footprints:R_0402_1005Metric, F.Cu at (157.6, 77.8)
- added U10: AP22615A_TSOT26, PC_Components_1:TSOT23-6, F.Cu at (71.0, 68.0)
- added U13: AP22615A_TSOT26, PC_Components_1:TSOT23-6, F.Cu at (88.0, 68.0)
- added U14: ESD204DQAR, PC_Components_1:USON-10_2.5x1mm_P0.5mm, F.Cu at (82.5, 69.4)
- added U19: TPS56C230, antmicro-footprints:QFN-20-1EP_3x3mm_P0.45mm_TPS56xxxx, F.Cu at (160.7, 76.8)
- added U21: TPS564247DRLR, antmicro-footprints:SOT-563, F.Cu at (169.9, 97.1)
- added U23: TLV73333PDBVT, antmicro-footprints:SOT-23-5, F.Cu at (160.5, 127.2)
- added U4: STM32G0B1RCT6, PC_ExtensionBoard:LQFP-64_L10.0-W10.0-P0.50-LS12.0-BL, F.Cu at (154.8, 118.2)
- added U49: INA219AIDCNR, antmicro-footprints:SOT-23-8, F.Cu at (152.1, 78.2)
- added U50: INA219AIDCNR, antmicro-footprints:SOT-23-8, F.Cu at (160.6, 94.5)
- added U8: ESD204DQAR, PC_Components_1:USON-10_2.5x1mm_P0.5mm, F.Cu at (76.5, 69.4)
- added U9: CH224K, PC_ExtensionBoard:ESSOP-10_L4.9-W3.9-P1.0-LS6.0-TL-EP, B.Cu at (155.3, 65.3)
- moved U2 2.00 mm to (63.2, 55.6)
Connections:
- U3 pad A88: unconnected-(U3I-PCIE_CLK+-PadA88) -> /PC_CoreBoard/PCIE_{REF}.CK+
- U3 pad A89: unconnected-(U3I-PCIE_CLK--PadA89) -> /PC_CoreBoard/PCIE_{REF}.CK-
Routing:
- net GND: track 0.00 -> 3.67 mm, vias 0 -> 4
- net /PC_CoreBoard/USBSS0.RX+: track 0.00 -> 1.51 mm
- net /PC_CoreBoard/USBSS0.RX-: track 0.00 -> 1.13 mm
Other:
- outline, holes or cut-outs redrawn
