File: PC_ExtensionBoard/PC_ExtensionBoard.kicad_pcb (KiCad board)
At the start: 6 copper layers, 128.2 x 98.2 mm, 269 parts, among them J100 Bus_M.2_2199230-2, J3 Conn_01x16_MountingPin, J4 Conn_01x02_Socket, J5 Conn_01x02_Socket, J6 Conn_01x04_Pin, J7 Conn_01x02_Socket, J8 Bus_M.2_1-2199230-6, Q10 2SK3018, Q11 2N7002, Q3 BSS138-7-F, Q4 SI7613DN-T1-GE3, Q7 BSS138-7-F, Q8 BSS138-7-F, Q9 2SK3018, SW1 K2-1808SN-A4SW, U1 HC-USB3.0-L168-WP, U10 AP22615A_TSOT26, U12 DC-528φ2.0(HY), U13 AP22615A_TSOT26, U14 ESD204DQAR, U15 AP22615A_TSOT26, U16 ESD204DQAR, U17 AP22615A_TSOT26, U18 ESD204DQAR, U19 TPS56C230, U2 10GHz, U20 TPS3840PL30DBVR, U21 TPS564247DRLR, U23 TLV73333PDBVT, U3 KBLH-E61_COMe_Type6_16U, U37 9DBL0651CKILF, U38 74AUP2G132, U4 STM32G0B1RCT6, U49 INA219AIDCNR, U5 TPAZ1023-04F, U50 INA219AIDCNR, U6 TPAZ1023-04F, U7 HC-USB3.0-L168-WP, U8 ESD204DQAR, U9 CH224K, Y1 Oscillator_32.768kHz_ECS_2520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

Commit message: DRC Bug fixes
Routing:
- net +12V: vias 82 -> 81
