File: PC_ExtensionBoard/USB.kicad_sch (KiCad schematic)
At the start: 88 parts, among them J1 Amphenol_RJE361882415, J2 Amphenol_RJE361882415, J4 Amphenol_RJE361882415, U1 HC-USB3.0-L168-WP, U10 AP22615A_TSOT26, U11 AP22615A_TSOT26, U12 ESD204DQAR, U13 AP22615A_TSOT26, U4 ESD204DQAR, U5 AP22615A_TSOT26, U6 ESD204DQAR, U7 AP22615A_TSOT26, U8 ESD204DQAR, U9 ESD204DQAR

Commit message: update schematic: add pattern
Parts:
- removed C10, C14: C_Pol_100u_10V_KEMET-T520-B, antmicro-footprints:C_Pol_EIA-B, symbol antmicroCapacitorspol:C_Pol_100u_10V_KEMET-T520-B
- removed C12, C13, C15, C6: C_1u_0402, antmicro-footprints:C_0402_1005Metric, symbol antmicroCapacitors0402:C_1u_0402
- removed C21, C24: C_100n_0402, antmicro-footprints:C_0402_1005Metric, symbol antmicroCapacitors0402:C_100n_0402
- removed C23, C25: C_22u_16V_0603, antmicro-footprints:C_0603_1608Metric, symbol antmicroCapacitors0603:C_22u_16V_0603
- removed D28, D29: TPD2E2U06_SC70, antmicro-footprints:SC70-3, symbol antmicroTVSDiodes:TPD2E2U06_SC70
- removed D4, D5: PESD5Z5_0F, antmicro-footprints:SOD-523, symbol antmicroTVSDiodes:PESD5Z5_0F
- removed J4: Amphenol_RJE361882415, antmicro-footprints:RJ45_RJE361882415, symbol antmicroModularConnectorsJacks:Amphenol_RJE361882415
- removed R15, R16: R_2k2_0402, antmicro-footprints:R_0402_1005Metric, symbol antmicroResistors0402:R_2k2_0402
- removed R31, R37, R42, R45: R_10k_0402, antmicro-footprints:R_0402_1005Metric, symbol antmicroResistors0402:R_10k_0402
- removed R34, R35, R40, R41, R43, R44, R47: R_0R_0402, antmicro-footprints:R_0402_1005Metric, symbol antmicroResistors0402:R_0R_0402
- removed U11, U13: AP22615A_TSOT26, antmicro-footprints:TSOT23-6, symbol antmicroPMICPowerDistributionSwitchesLoadDrivers:AP22615A_TSOT26
- removed U12, U9: ESD204DQAR, antmicro-footprints:USON-10_2.5x1mm_P0.5mm, symbol antmicroTVSDiodes:ESD204DQAR
- added C13, C15, C34, C35, C36: C_100n_0402, antmicro-footprints:C_0402_1005Metric, symbol antmicroCapacitors0402:C_100n_0402
- added C14: C_1n_1210_2kV, antmicro-footprints:C_1210_3225Metric, symbol antmicroCapacitorsmisc:C_1n_1210_2kV
- added unit 1 of J1
- added R1, R2, R3, R4, R5, R6: R_0R_0402, antmicro-footprints:R_0402_1005Metric, symbol antmicroResistors0402:R_0R_0402
- added R10, R330, R331, R7, R8, R9: R_470R_0402, antmicro-footprints:R_0402_1005Metric, symbol antmicroResistors0402:R_470R_0402
- added R11: R_330R_0402, antmicro-footprints:R_0402_1005Metric, symbol antmicroResistors0402:R_330R_0402
- added R16, R43, R44, R45: R_75R_0402, antmicro-footprints:R_0402_1005Metric, symbol antmicroResistors0402:R_75R_0402
- added RJ1: DS1128-09-S8B8S, ACLAB:RJ45-TH_DS1128-09-S8B8S, symbol ACLAB_Symbol:root_0_DS1128-09-S8B8S_
- added T1, T2, T3, T4: Choke_SRF2012A-801Y, antmicro-footprints:Choke_0805_2012Metric, symbol antmicroCommonModeChokes:Choke_SRF2012A-801Y
- added T5, T6, T7, T8: Trans_SM453229-381N7Y, antmicro-footprints:Trans_Eth_4.7x3.3mm, symbol antmicroInterfaceDriversReceiversTransceivers:Trans_SM453229-381N7Y
- added U2: 10GHz, ACLAB:SMA-TH_SMA-KWE, symbol ACLAB_Symbol:root_0_SMA-KWE_C20415790_
- added unit 2 of USB1
- added USB2: HC-USB3.0-L175-2X1-P, ACLAB:USB-A-TH_H181-AF2R06-12ALCR, symbol ACLAB_Symbol:root_0_HC-USB3.0-L175-2X1-P_
- C11: footprint antmicro-footprints:C_0402_1005Metric -> (none); Author Antmicro -> (none); LCSC (none) -> C2182694
- C5: footprint antmicro-footprints:C_0402_1005Metric -> Capacitor_SMD:C_0402_1005Metric; Author Antmicro -> (none); LCSC (none) -> C2182694
- C7: footprint antmicro-footprints:C_Pol_EIA-B -> (none); Author Antmicro -> (none); LCSC (none) -> C600583
- D27: footprint antmicro-footprints:SC70-3 -> (none); Author Antmicro -> (none); LCSC (none) -> C1855726
- D3: footprint antmicro-footprints:SOD-523 -> (none); Author Antmicro -> (none); LCSC (none) -> C552600
- R14: footprint antmicro-footprints:R_0402_1005Metric -> (none); Author Antmicro -> (none); LCSC (none) -> C2076845
- R36: footprint antmicro-footprints:R_0402_1005Metric -> (none); Author Antmicro -> (none); LCSC (none) -> C202396
- R38, R39: footprint antmicro-footprints:R_0402_1005Metric -> (none); Author Antmicro -> (none); LCSC (none) -> C242160
- U10: footprint antmicro-footprints:TSOT23-6 -> (none); Author Antmicro -> (none); LCSC (none) -> C2680357
- U8: footprint antmicro-footprints:USON-10_2.5x1mm_P0.5mm -> (none); Author Antmicro -> (none); LCSC (none) -> C553132
Connections:
- net +3V3: now also R10.2, R7.2, R8.2, R9.2
- net FLG_1B: no longer R46.2
- net GND: now also C13.2, C14.1, C15.2, C34.2, C35.2, C36.2, R11.2, R330.1, R331.1, USB1.13 (GND), USB1.16 (GND_DRAIN), USB1.20 (GND); no longer USB1.13 (GND), USB1.20 (GND), USB1.4 (GND)
- net P0_D+: now also USB1.11 (D-); no longer USB1.11 (D-)
- net P0_D-: now also USB1.12 (D+); no longer USB1.12 (D+)
- net P0_VBUS: now also USB1.10 (VBUS); no longer USB1.10 (VBUS)
- net P1_D+: no longer USB1.2 (D-)
- net P1_D-: no longer USB1.3 (D+)
- net P1_VBUS: no longer USB1.1 (VBUS)
- net USBSS_0.RX+: now also USB1.15 (SSRX+); no longer USB1.15 (SSRX+)
- net USBSS_0.RX-: now also USB1.14 (SSRX-); no longer USB1.14 (SSRX-)
- net USBSS_0.TX+: now also USB1.18 (SSTX+); no longer USB1.18 (SSTX+)
- net USBSS_0.TX-: now also USB1.17 (SSTX-); no longer USB1.17 (SSTX-)
- net USBSS_1.RX+: no longer USB1.6 (SSRX+)
- net USBSS_1.RX-: no longer USB1.5 (SSRX-)
- net USBSS_1.TX+: no longer USB1.9 (SSTX+)
- net USBSS_1.TX-: no longer USB1.8 (SSTX-)
- net FLG_0 renamed USB_0_1_OC#
- net FLG_1: no longer names the net of R46.1
- net FLG_1: now also C15.1, C34.1, C35.1, C36.1, T5.3, T6.3, T7.3, T8.3
- new net: R44.2, T7.5
- new net: J1.D3 (LED_D3), R3.2, R6.2, R8.1
- new net: J1.D1 (LED_D1), R1.2, R331.2, R7.1
- new net: C14.2, R16.1, R43.1, R44.1, R45.1
- new net: J1.D2 (LED_D2), R2.2, R330.2, R9.1
- new net: J1.D4 (LED_D4), R10.1, R4.2, R5.2
- new net: R45.2, T8.5
- new net: R16.2, T5.5
- new net: R43.2, T6.5
- new net DA+: J1.1, T1.2
- new net DA-: J1.2, T1.3
- new net DA_FL+: T1.1, T5.1
- new net DA_FL-: T1.4, T5.2
- new net DB+: J1.3, T2.2
- new net DB-: J1.6, T2.3
- new net DB_FL+: T2.1, T6.1
- new net DB_FL-: T2.4, T6.2
- new net DC+: J1.4, T3.2
- new net DC-: J1.5, T3.3
- new net DC_FL+: T3.1, T7.1
- new net DC_FL-: T3.4, T7.2
- new net DD+: J1.7, T4.2
- new net DD-: J1.8, T4.3
- new net DD_FL+: T4.1, T8.1
- new net DD_FL-: T4.4, T8.2
- new net GbE.CTREF: R46.2
- new net GbE.MDI0+: T5.6
- new net GbE.MDI0-: T5.7
- new net GbE.MDI1+: T6.6
- new net GbE.MDI1-: T6.7
- new net GbE.MDI2+: T7.6
- new net GbE.MDI2-: T7.7
- new net GbE.MDI3+: T8.6
- new net GbE.MDI3-: T8.7
- new net SH: C13.1, J1.MP, R11.1
- new net ~{GBE0_ACT}: R1.1, R2.1
- new net ~{GBE0_LINK_1000}: R3.1, R5.1
- new net ~{GBE0_LINK}: R4.1, R6.1
Other:
- note added: "Dual_USB3.0_PORT_BACK_SIDE"
- note added: "GbE RJ45"
- note added: "LED polarity missing from datasheet so we're ready for both"
- note added: "USB3.0_PORT_FRONT"
- moved on the sheet: C11, C18, C22, C5, C7, D27, D3, R14, R30, R32, R33, R36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

Commit message: update Schematic
Parts:
- removed C1, C2, C8, C9: C_1u_0402, antmicro-footprints:C_0402_1005Metric, symbol antmicroCapacitors0402:C_1u_0402
- removed C16, C17: C_100n_0402, antmicro-footprints:C_0402_1005Metric, symbol antmicroCapacitors0402:C_100n_0402
- removed C19, C20: C_22u_16V_0603, antmicro-footprints:C_0603_1608Metric, symbol antmicroCapacitors0603:C_22u_16V_0603
- removed C3, C4: C_Pol_100u_10V_KEMET-T520-B, antmicro-footprints:C_Pol_EIA-B, symbol antmicroCapacitorspol:C_Pol_100u_10V_KEMET-T520-B
- removed D1, D2: PESD5Z5_0F, antmicro-footprints:SOD-523, symbol antmicroTVSDiodes:PESD5Z5_0F
- removed D25, D26: TPD2E2U06_SC70, antmicro-footprints:SC70-3, symbol antmicroTVSDiodes:TPD2E2U06_SC70
- removed unit 2 of J1
- removed J2: Amphenol_RJE361882415, antmicro-footprints:RJ45_RJE361882415, symbol antmicroModularConnectorsJacks:Amphenol_RJE361882415
- removed R12, R13: R_2k2_0402, antmicro-footprints:R_0402_1005Metric, symbol antmicroResistors0402:R_2k2_0402
- removed R18, R19, R24, R25: R_10k_0402, antmicro-footprints:R_0402_1005Metric, symbol antmicroResistors0402:R_10k_0402
- removed R20, R21, R22, R23, R26, R27, R28, R29: R_0R_0402, antmicro-footprints:R_0402_1005Metric, symbol antmicroResistors0402:R_0R_0402
- removed U4, U6: ESD204DQAR, antmicro-footprints:USON-10_2.5x1mm_P0.5mm, symbol antmicroTVSDiodes:ESD204DQAR
- removed U5, U7: AP22615A_TSOT26, antmicro-footprints:TSOT23-6, symbol antmicroPMICPowerDistributionSwitchesLoadDrivers:AP22615A_TSOT26
- removed USB2: HC-USB3.0-L175-2X1-P, ACLAB:USB-A-TH_H181-AF2R06-12ALCR, symbol ACLAB_Symbol:root_0_HC-USB3.0-L175-2X1-P_
- added C10, C41: C_Pol_100u_10V_KEMET-T520-B, PC_Components_1:C_Pol_EIA-B, symbol antmicroCapacitorspol:C_Pol_100u_10V_KEMET-T520-B
- added C12, C38: C_1u_0402, PC_Components_1:C_0402_1005Metric, symbol antmicroCapacitors0402:C_1u_0402
- added C31, C33: C_22u_16V_0603, PC_Components_1:C_0603_1608Metric, symbol antmicroCapacitors0603:C_22u_16V_0603
- added C32, C37: C_100n_0402, PC_Components_1:C_0402_1005Metric, symbol antmicroCapacitors0402:C_100n_0402
- added C42, C6: C_1u_0402, Capacitor_SMD:C_0402_1005Metric, symbol antmicroCapacitors0402:C_1u_0402
- added D20, D9: PESD5Z5_0F, PC_Components_1:SOD-523, symbol antmicroTVSDiodes:PESD5Z5_0F
- added D28, D29: TPD2E2U06_SC70, PC_Components_1:SC70-3, symbol antmicroTVSDiodes:TPD2E2U06_SC70
- added R58, R59, R61, R62, R65, R66, R68, R69: R_0R_0402, PC_Components_1:C_0402_1005Metric, symbol antmicroResistors0402:R_0R_0402
- added R60, R63, R67, R70: R_10k_0402, PC_Components_1:C_0402_1005Metric, symbol antmicroResistors0402:R_10k_0402
- added R64, R71: R_2k2_0402, PC_Components_1:C_0402_1005Metric, symbol antmicroResistors0402:R_2k2_0402
- added U13, U15: AP22615A_TSOT26, PC_Components_1:TSOT23-6, symbol antmicroPMICPowerDistributionSwitchesLoadDrivers:AP22615A_TSOT26
- added U14, U16: ESD204DQAR, PC_Components_1:USON-10_2.5x1mm_P0.5mm, symbol antmicroTVSDiodes:ESD204DQAR
- C11: footprint (none) -> PC_Components_1:C_0402_1005Metric; License Apache-2.0 -> (none); Manufacturer TDK -> (none); Public False -> (none)
- C18: footprint antmicro-footprints:C_0402_1005Metric -> PC_Components_1:C_0402_1005Metric; Author Antmicro -> (none); LCSC (none) -> C85960; License Apache-2.0 -> (none); Public False -> (none)
- C22: footprint antmicro-footprints:C_0603_1608Metric -> PC_Components_1:C_0603_1608Metric; Author Antmicro -> (none); LCSC (none) -> C2762594; License Apache-2.0 -> (none); Public False -> (none)
- C5: License Apache-2.0 -> (none); MPN C1005X6S1A105K050BC -> (none); Public False -> (none)
- C7: footprint (none) -> PC_Components_1:C_Pol_EIA-B; Dielectric template_dielectric -> (none); License Apache-2.0 -> (none); Manufacturer KEMET -> (none); Public False -> (none)
- D27: footprint (none) -> PC_Components_1:SC70-3; License Apache-2.0 -> (none); Manufacturer Texas Instruments -> (none)
- D3: footprint (none) -> PC_Components_1:SOD-523; License Apache-2.0 -> (none); Manufacturer Nexperia -> (none); Public False -> (none)
- R14, R36: footprint (none) -> PC_Components_1:C_0402_1005Metric; License Apache-2.0 -> (none); Manufacturer Bourns -> (none); Public False -> (none)
- R30: footprint antmicro-footprints:R_0402_1005Metric -> PC_Components_1:C_0402_1005Metric; Author Antmicro -> (none); License Apache-2.0 -> (none); Manufacturer Bourns -> (none); Public False -> (none)
- R32, R33: footprint antmicro-footprints:R_0402_1005Metric -> PC_Components_1:C_0402_1005Metric; Author Antmicro -> (none); LCSC (none) -> C242160; License Apache-2.0 -> (none); Public False -> (none)
- R38: footprint (none) -> PC_Components_1:C_0402_1005Metric; License Apache-2.0 -> (none); Manufacturer Panasonic -> (none); Public False -> (none)
- R39: footprint (none) -> PC_Components_1:C_0402_1005Metric; License Apache-2.0 -> (none); Public False -> (none)
- U10: footprint (none) -> PC_Components_1:TSOT23-6; License Apache-2.0 -> (none); Manufacturer Diodes Incorporated -> (none)
- U8: footprint (none) -> PC_Components_1:USON-10_2.5x1mm_P0.5mm; License Apache-2.0 -> (none)
- USB1: footprint ACLAB:USB-A-TH_H181-AF2R06-12ALCR -> PC_ExtensionBoard:USB-A-TH_H181-AF2R06-12ALCR; CONTRIBUTOR lcsc -> (none); JLCPCB PART CLASS Extended Part -> (none); MANUFACTURER HC(虹成电子) -> (none); MANUFACTURER PART HC-USB3.0-L175-2X1-P -> (none); SPICEPRE U -> (none); SPICESYMBOLNAME HC-USB3.0-L175-2X1-P -> (none); SUPPLIER LCSC -> (none)
Connections:
- net +3V3: now also R60.2, R63.2, R67.2, R70.2
- net +5V: now also C31.2, C32.2, C33.2, C37.2, U13.6 (IN), U15.6 (IN)
- net EN_1B: now also R58.2, R60.1, U13.4 (EN)
- net FLG_1B: now also R59.2, R63.1, U13.3 (FLG)
- net GND: now also U1.10 (SH), U1.4 (GND), U1.7 (GND_DRAN), USB1.4 (GND), USB1.7 (GND_DRAIN), C10.2, C12.1, C31.1, C32.1, C33.1, C37.1, C38.1, C41.2, C42.1, C6.1, D20.2 (A), D28.3, D29.3, D9.2 (A), R64.1, R71.1, U13.2 (GND), U14.3, U14.8, U15.2 (GND), U16.3, U16.8
- net P0_D+: now also USB1.12 (D+); no longer USB1.11 (D-)
- net P0_D-: now also USB1.11 (D-); no longer USB1.12 (D+)
- net P1_D+: now also USB1.3 (D+), D28.2, R62.2
- net P1_D-: now also USB1.2 (D-), D28.1, R61.2
- net P1_ISET: now also R64.2, U13.5 (ISET)
- net P1_VBUS: now also USB1.1 (VBUS), C10.1, C12.2, C6.2, D9.1 (C), U13.1 (OUT)
- net USBSS_1.RX+: now also USB1.6 (SSRX+), U14.2, U14.9
- net USBSS_1.RX-: now also USB1.5 (SSRX-), U14.1, U14.10
- net USBSS_1.TX+: now also USB1.9 (SSTX+), U14.5, U14.6
- net USBSS_1.TX-: now also USB1.8 (SSTX-), U14.4, U14.7
- net USB_0_1_OC#: now also R59.1
- net USB_1.D+: now also R62.1
- net USB_1.D-: now also R61.1
- net P2_VBUS: now reaches U1.1 (VBUS)
- net P2_VBUS: now also C38.2, C41.1, C42.2, D20.1 (C), U15.1 (OUT)
- net P2_D-: now reaches U1.2 (D-)
- net P2_D-: now also D29.1, R68.2
- net P2_D+: now reaches U1.3 (D+)
- net P2_D+: now also D29.2, R69.2
- net USBSS_2.RX-: now reaches U1.5 (SSRX-)
- net USBSS_2.RX-: now also U16.1, U16.10
- net USBSS_2.RX+: now reaches U1.6 (SSRX+)
- net USBSS_2.RX+: now also U16.2, U16.9
- net USBSS_2.TX-: now reaches U1.8 (SSTX-)
- net USBSS_2.TX-: now also U16.4, U16.7
- net USBSS_2.TX+: now reaches U1.9 (SSTX+)
- net USBSS_2.TX+: now also U16.5, U16.6
- new net EN_1: R58.1
- new net EN_2: R65.1
- new net EN_2B: R65.2, R67.1, U15.4 (EN)
- new net FLG_2B: R66.2, R70.1, U15.3 (FLG)
- new net P2_ISET: R71.2, U15.5 (ISET)
- new net USB_2.D+: R69.1
- new net USB_2.D-: R68.1
- new net USB_2_3_OC#: R66.1
Other:
- note added: "USB_C_3.0_PORT_BACK"
- note removed: "USB 3.0"
- moved on the sheet: C13, C14, C15, C34, C35, C36, J1A, PJ1, R1, R10, R11, R16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

Commit message: refactor project
Parts:
- C10, C41, C7: symbol antmicroCapacitorspol:C_Pol_100u_10V_KEMET-T520-B -> A_PC_ExtensionBoard:C_Pol_100u_10V_KEMET-T520-B
- C11, C12, C38, C42, C5, C6: symbol antmicroCapacitors0402:C_1u_0402 -> A_PC_ExtensionBoard:C_1u_0402
- C13, C15, C18, C32, C34, C35, C36, C37: symbol antmicroCapacitors0402:C_100n_0402 -> A_PC_ExtensionBoard:C_100n_0402
- C14: symbol antmicroCapacitorsmisc:C_1n_1210_2kV -> A_PC_ExtensionBoard:C_1n_1210_2kV
- C22, C31, C33: symbol antmicroCapacitors0603:C_22u_16V_0603 -> A_PC_ExtensionBoard:C_22u_16V_0603
- D20, D3, D9: symbol antmicroTVSDiodes:PESD5Z5_0F -> A_PC_ExtensionBoard:PESD5Z5_0F
- D27, D28, D29: symbol antmicroTVSDiodes:TPD2E2U06_SC70 -> A_PC_ExtensionBoard:TPD2E2U06_SC70
- J1: symbol antmicroModularConnectorsJacks:Amphenol_RJE361882415 -> A_PC_ExtensionBoard:Amphenol_RJE361882415
- PJ1: symbol ACLAB_Symbol:root_0_PJ-327A_ -> A_PC_ExtensionBoard:Audio_PJ-327A_
- R1, R2, R3, R4, R46, R5, R6: symbol antmicroResistors0402:R_0R_0402 -> A_PC_ExtensionBoard:R_0R_0402
- R10, R330, R331, R7, R8, R9: symbol antmicroResistors0402:R_470R_0402 -> A_PC_ExtensionBoard:R_470R_0402
- R11: symbol antmicroResistors0402:R_330R_0402 -> A_PC_ExtensionBoard:R_330R_0402
- R14, R64, R71: symbol antmicroResistors0402:R_2k2_0402 -> A_PC_ExtensionBoard:R_2k2_0402
- R16, R43, R44, R45: symbol antmicroResistors0402:R_75R_0402 -> A_PC_ExtensionBoard:R_75R_0402
- R30, R36, R60, R63, R67, R70: footprint PC_Components_1:C_0402_1005Metric -> antmicro-footprints:R_0402_1005Metric; symbol antmicroResistors0402:R_10k_0402 -> A_PC_ExtensionBoard:R_10k_0402; Author (none) -> Antmicro; License (none) -> Apache-2.0; Manufacturer (none) -> Bourns; Public (none) -> False
- R32, R33, R39, R58, R61, R62, R65, R68, R69: footprint PC_Components_1:C_0402_1005Metric -> antmicro-footprints:R_0402_1005Metric; symbol antmicroResistors0402:R_0R_0402 -> A_PC_ExtensionBoard:R_0R_0402; Author (none) -> Antmicro; License (none) -> Apache-2.0; Public (none) -> False
- R38, R59, R66: footprint PC_Components_1:C_0402_1005Metric -> antmicro-footprints:R_0402_1005Metric; symbol antmicroResistors0402:R_0R_0402 -> A_PC_ExtensionBoard:R_0R_0402; Author (none) -> Antmicro; License (none) -> Apache-2.0; Manufacturer (none) -> Panasonic; Public (none) -> False
- RJ1: symbol ACLAB_Symbol:root_0_DS1128-09-S8B8S_ -> A_PC_ExtensionBoard:RJ45_DS1128-09-S8B8S_
- T1, T2, T3, T4: symbol antmicroCommonModeChokes:Choke_SRF2012A-801Y -> A_PC_ExtensionBoard:Choke_SRF2012A-801Y
- T5, T6, T7, T8: symbol antmicroInterfaceDriversReceiversTransceivers:Trans_SM453229-381N7Y -> A_PC_ExtensionBoard:Trans_SM453229-381N7Y
- U1: symbol ACLAB_Symbol:root_0_HC-USB3.0-L168-WP_ -> A_PC_ExtensionBoard:HC-USB3.0-L168-WP
- U10, U13, U15: symbol antmicroPMICPowerDistributionSwitchesLoadDrivers:AP22615A_TSOT26 -> A_PC_ExtensionBoard:AP22615A_TSOT26
- U14, U16, U8: symbol antmicroTVSDiodes:ESD204DQAR -> A_PC_ExtensionBoard:ESD204DQAR
- U2: symbol ACLAB_Symbol:root_0_SMA-KWE_C20415790_ -> A_PC_ExtensionBoard:Antenna_SMA-KWE_C20415790_
- USB1: symbol ACLAB_Symbol:root_0_HC-USB3.0-L175-2X1-P_ -> A_PC_ExtensionBoard:HC-USB3.0-L175-2X1-P
- USBC1, USBC2: symbol ACLAB_Symbol:root_0_TYPE-C-31-M-12_ -> A_PC_ExtensionBoard:TYPE-C-31-M-12
Connections:
- net +3V3 renamed +3.3V

Commit message: re-link symbol
Parts:
- removed C13, C15, C34, C35, C36: C_100n_0402, antmicro-footprints:C_0402_1005Metric, symbol A_PC_ExtensionBoard:C_100n_0402
- removed C14: C_1n_1210_2kV, antmicro-footprints:C_1210_3225Metric, symbol A_PC_ExtensionBoard:C_1n_1210_2kV
- removed J1: Amphenol_RJE361882415, antmicro-footprints:RJ45_RJE361882415, symbol A_PC_ExtensionBoard:Amphenol_RJE361882415
- removed PJ1: PJ-327A, ACLAB:AUDIO-IN-SMD_PJ-327A_C22355751, symbol A_PC_ExtensionBoard:Audio_PJ-327A_
- removed R1, R2, R3, R4, R46, R5, R6: R_0R_0402, antmicro-footprints:R_0402_1005Metric, symbol A_PC_ExtensionBoard:R_0R_0402
- removed R10, R330, R331, R7, R8, R9: R_470R_0402, antmicro-footprints:R_0402_1005Metric, symbol A_PC_ExtensionBoard:R_470R_0402
- removed R11: R_330R_0402, antmicro-footprints:R_0402_1005Metric, symbol A_PC_ExtensionBoard:R_330R_0402
- removed R16, R43, R44, R45: R_75R_0402, antmicro-footprints:R_0402_1005Metric, symbol A_PC_ExtensionBoard:R_75R_0402
- removed RJ1: DS1128-09-S8B8S, ACLAB:RJ45-TH_DS1128-09-S8B8S, symbol A_PC_ExtensionBoard:RJ45_DS1128-09-S8B8S_
- removed T1, T2, T3, T4: Choke_SRF2012A-801Y, antmicro-footprints:Choke_0805_2012Metric, symbol A_PC_ExtensionBoard:Choke_SRF2012A-801Y
- removed T5, T6, T7, T8: Trans_SM453229-381N7Y, antmicro-footprints:Trans_Eth_4.7x3.3mm, symbol A_PC_ExtensionBoard:Trans_SM453229-381N7Y
- removed U2: 10GHz, ACLAB:SMA-TH_SMA-KWE, symbol A_PC_ExtensionBoard:Antenna_SMA-KWE_C20415790_
- added C21, C23: C_100n_0402, PC_Components_1:C_0402_1005Metric, symbol A_PC_ExtensionBoard:C_100n_0402
- added R17: R_330R_0402, PC_Components_1:R_0402_1005Metric, symbol A_PC_ExtensionBoard:R_330R_0402
- added R332, R333: R_470R_0402, PC_Components_1:R_0402_1005Metric, symbol A_PC_ExtensionBoard:R_470R_0402
- added RJ1: HR911130A, C54408:RJ45-TH_HR911130A, symbol A_PC_ExtensionBoard:HR911130A
- R30, R32, R33, R36, R38, R39, R58, R59, R60, R61, R62, R63, R65, R66, R67, R68, R69, R70: footprint antmicro-footprints:R_0402_1005Metric -> PC_Components_1:R_0402_1005Metric
- USB1: footprint PC_ExtensionBoard:USB-A-TH_H181-AF2R06-12ALCR -> PC_Components_1:USB-A-TH_H181-AF2R06-12ALCR
Connections:
- net +3.3V: now also R332.2, R333.2
- net GND: now also C21.2, C23.2, R17.2
- net GbE.CTREF: now also C21.1, RJ1.P1
- net GbE.MDI0+: now also RJ1.P2 (MDI0+)
- net GbE.MDI0-: now also RJ1.P3 (MDI0-)
- net GbE.MDI1+: now also RJ1.P4 (MDI1+)
- net GbE.MDI1-: now also RJ1.P7 (MDI1-)
- net GbE.MDI2+: now also RJ1.P5 (MDI2+)
- net GbE.MDI2-: now also RJ1.P6 (MDI2-)
- net GbE.MDI3+: now also RJ1.P8 (MDI3+)
- net GbE.MDI3-: now also RJ1.P9 (MDI3-)
- net ~{GBE0_ACT}: now also RJ1.12
- net ~{GBE0_LINK_1000}: now also RJ1.13
- new net: R332.1, RJ1.11
- new net: R333.1, RJ1.14
- new net: C23.1, R17.1, RJ1.P10, RJ1.SHIELD0, RJ1.SHIELD1
Other:
- note added: "RJ45"
- note removed: "GbE RJ45"
- note removed: "LED polarity missing from datasheet so we're ready for both"

Commit message: update LCSC for HDMI
Parts:
- removed USBC1, USBC2: TYPE-C-31-M-12, ACLAB:USB-C_SMD-TYPE-C-31-M-12_1, symbol A_PC_ExtensionBoard:TYPE-C-31-M-12
- added Audio1: PJ-393-7A, PC_Components_1:AUDIO-SMD_PJ-393-7A, symbol A_PC_ExtensionBoard:PJ-393-7A
- added C34: C_22u_16V_0603, PC_Components_1:C_0603_1608Metric, symbol A_PC_ExtensionBoard:C_22u_16V_0603
- added C35, C36, C43: C_100n_0402, PC_Components_1:C_0402_1005Metric, symbol A_PC_ExtensionBoard:C_100n_0402
- added C44, C60, C63: C_1u_0402, PC_Components_1:C_0402_1005Metric, symbol A_PC_ExtensionBoard:C_1u_0402
- added C46: C_Pol_100u_10V_KEMET-T520-B, PC_Components_1:C_Pol_EIA-B, symbol A_PC_ExtensionBoard:C_Pol_100u_10V_KEMET-T520-B
- added C47: C_1u_0402, Capacitor_SMD:C_0402_1005Metric, symbol A_PC_ExtensionBoard:C_1u_0402
- added C65: C_10u_0402, PC_Components_1:C_0402_1005Metric, symbol A_PC_ExtensionBoard:C_1u_0402
- added D22: PESD5Z5_0F, PC_Components_1:SOD-523, symbol A_PC_ExtensionBoard:PESD5Z5_0F
- added D30: TPD2E2U06_SC70, PC_Components_1:SC70-3, symbol A_PC_ExtensionBoard:TPD2E2U06_SC70
- added R72, R73, R75, R76: R_0R_0402, PC_Components_1:R_0402_1005Metric, symbol A_PC_ExtensionBoard:R_0R_0402
- added R74, R77: R_10k_0402, PC_Components_1:R_0402_1005Metric, symbol A_PC_ExtensionBoard:R_10k_0402
- added R78: R_2k2_0402, PC_Components_1:C_0402_1005Metric, symbol A_PC_ExtensionBoard:R_2k2_0402
- added R79: R_20K_0402, PC_Components_1:R_0402_1005Metric, symbol A_PC_ExtensionBoard:R_0R_0402
- added U11: ALC662, Package_QFP:LQFP-48-1EP_7x7mm_P0.5mm_EP3.6x3.6mm, symbol A_PC_ExtensionBoard:ALC662
- added U17: AP22615A_TSOT26, PC_Components_1:TSOT23-6, symbol A_PC_ExtensionBoard:AP22615A_TSOT26
- added U18: ESD204DQAR, PC_Components_1:USON-10_2.5x1mm_P0.5mm, symbol A_PC_ExtensionBoard:ESD204DQAR
- added U7: HC-USB3.0-L168-WP, ACLAB:USB-TH_USB3.0-A, symbol A_PC_ExtensionBoard:HC-USB3.0-L168-WP
- C21, C23: LCSC (none) -> C85960
- R17: LCSC (none) -> C2077069
- R332, R333: LCSC (none) -> C2077077
Connections:
- net +3.3V: now also C36.1, C63.2, R74.2, R77.2, U11.1 (DVDD), U11.9 (DVDD-IO)
- net +5V: now also C34.2, C35.1, C43.2, C60.2, U11.25 (AVDD1), U11.38 (AVDD2), U17.6 (IN)
- net GND: now also Audio1.4, C34.1, C35.2, C36.2, C43.1, C44.1, C46.2, C47.1, C60.1, C63.1, C65.1, D22.2 (A), D30.3, R78.1, R79.1, U11.26 (AVSS1), U11.4 (DVSS), U11.42 (AVSS2), U11.7 (DVSS), U17.2 (GND), U18.3, U18.8, U7.10 (SH), U7.4 (GND), U7.7 (GND_DRAN)
- net USB_2_3_OC#: now also R73.1
- new net: Audio1.2, U11.35 (FRONT-L)
- new net: Audio1.3, U11.36 (FRONT-R)
- new net: Audio1.5, U11.13 (Sense_A)
- new net: C65.2, U11.27 (VREF)
- new net: R79.2, U11.40 (JDREF)
- new net BITCLK: U11.6 (BITCLK)
- new net EN_3: R72.1
- new net EN_3B: R72.2, R74.1, U17.4 (EN)
- new net FLG_3B: R73.2, R77.1, U17.3 (FLG)
- new net MIC1-VREF0-L: Audio1.1, U11.21 (MIC1-L), U11.28 (MIC1-VREFO-L)
- new net P3_D+: D30.2, R76.2, U7.3 (D+)
- new net P3_D-: D30.1, R75.2, U7.2 (D-)
- new net P3_ISET: R78.2, U17.5 (ISET)
- new net P3_VBUS: C44.2, C46.1, C47.2, D22.1 (C), U17.1 (OUT), U7.1 (VBUS)
- new net RST: U11.11 (RESET#)
- new net SDIN0: U11.8 (SDATA-IN)
- new net SDOUT: U11.5 (SDATA-OUT)
- new net SYNC: U11.10 (SYNC)
- new net USBSS_3.RX+: U18.2, U18.9, U7.6 (SSRX+)
- new net USBSS_3.RX-: U18.1, U18.10, U7.5 (SSRX-)
- new net USBSS_3.TX+: U18.5, U18.6, U7.9 (SSTX+)
- new net USBSS_3.TX-: U18.4, U18.7, U7.8 (SSTX-)
- new net USB_3.D+: R76.1
- new net USB_3.D-: R75.1
- no-connect marks 0 -> 25
Other:
- note added: "ALC662"
- note removed: "USB_C_3.0_PORT_BACK"
