File: PC_ExtensionBoard/M.2 Key E.kicad_sch (KiCad schematic)
At the start: 18 parts, among them J100 Bus_M.2_2199230-2, U2 10GHz

Commit message: bug fixes
Connections:
- net PCIE_{REF3}.CK+ renamed PCIE_REF3.CK+
- net PCIE_{REF3}.CK- renamed PCIE_REF3.CK-
- net PCIe_{B1x2}.RX0+ renamed PCIe_B1x2.RX0+
- net PCIe_{B1x2}.RX0- renamed PCIe_B1x2.RX0-
- net PCIe_{B1x2}.TX0+ renamed PCIe_B1x2.TX0+
- net PCIe_{B1x2}.TX0- renamed PCIe_B1x2.TX0-
Changed lines of the file:
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@@
 		)
 	)
-	(label "PCIe_{B1x2}.RX1-"
+	(label "PCIe_B1x2.RX1-"
 		(at 62.23 100.33 180)
 		(effects
@@
 		)
 	)
-	(label "PCIe_{B1x2}.RX0+"
+	(label "PCIe_B1x2.RX0+"
 		(at 45.72 80.01 0)
 		(effects
@@
 		)
 	)
-	(label "PCIe_{B1x2}.TX0+"
+	(label "PCIe_B1x2.TX0+"
 		(at 45.72 72.39 0)
 		(effects
@@
 		)
 	)
-	(label "PCIE_{REF3}.CK+"
+	(label "PCIE_REF3.CK+"
 		(at 63.5 64.77 0)
 		(effects
@@
 		)
 	)
-	(label "PCIe_{B1x2}.RX1+"
+	(label "PCIe_B1x2.RX1+"
 		(at 62.23 97.79 180)
 		(effects
@@
 		)
 	)
-	(label "PCIe_{B1x2}.TX1+"
+	(label "PCIe_B1x2.TX1+"
 		(at 60.96 90.17 180)
 		(effects
@@
 		)
 	)
-	(label "PCIe_{B1x2}.RX0-"
+	(label "PCIe_B1x2.RX0-"
 		(at 45.72 82.55 0)
 		(effects
@@
 		)
 	)
-	(label "PCIE_{REF3}.CK-"
+	(label "PCIE_REF3.CK-"
 		(at 63.5 67.31 0)
 		(effects
@@
 		)
 	)
-	(label "PCIe_{B1x2}.TX0-"
+	(label "PCIe_B1x2.TX0-"
 		(at 45.72 74.93 0)
 		(effects
@@
 		)
 	)
-	(label "PCIe_{B1x2}.TX1-"
+	(label "PCIe_B1x2.TX1-"
 		(at 62.23 92.71 180)
 		(effects
@@
 		)
 	)
-	(hierarchical_label "PCIE_{REF3}{PCIe_{REF}}"
+	(hierarchical_label "PCIE_REF3{PCIe_REF}"
 		(shape input)
 		(at 36.83 59.69 180)
@@
 		)
 	)
-	(hierarchical_label "PCIe_{B1x2}{PCIe}"
+	(hierarchical_label "PCIe_B1x2{PCIe}"
 		(shape input)
 		(at 36.83 67.31 180)
