File: PC_ExtensionBoard/M.2 Key M #1.kicad_sch (KiCad schematic)
At the start: 16 parts, among them J8 Bus_M.2_1-2199230-6

Commit message: bug fixes
Connections:
- net PCIE_{REF0}.CK+ renamed PCIE_REF0.CK+
- net PCIE_{REF0}.CK- renamed PCIE_REF0.CK-
- net PCIe_{B1x4}.RX0+ renamed PCIe_B1x4.RX0+
- net PCIe_{B1x4}.RX0- renamed PCIe_B1x4.RX0-
- net PCIe_{B1x4}.RX1+ renamed PCIe_B1x4.RX1+
- net PCIe_{B1x4}.RX1- renamed PCIe_B1x4.RX1-
- net PCIe_{B1x4}.RX2+ renamed PCIe_B1x4.RX2+
- net PCIe_{B1x4}.RX2- renamed PCIe_B1x4.RX2-
- net PCIe_{B1x4}.RX3+ renamed PCIe_B1x4.RX3+
- net PCIe_{B1x4}.RX3- renamed PCIe_B1x4.RX3-
- net PCIe_{B1x4}.TX0+ renamed PCIe_B1x4.TX0+
- net PCIe_{B1x4}.TX0- renamed PCIe_B1x4.TX0-
- net PCIe_{B1x4}.TX1+ renamed PCIe_B1x4.TX1+
- net PCIe_{B1x4}.TX1- renamed PCIe_B1x4.TX1-
- net PCIe_{B1x4}.TX2+ renamed PCIe_B1x4.TX2+
- net PCIe_{B1x4}.TX2- renamed PCIe_B1x4.TX2-
- net PCIe_{B1x4}.TX3+ renamed PCIe_B1x4.TX3+
- net PCIe_{B1x4}.TX3- renamed PCIe_B1x4.TX3-
Changed lines of the file:
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@@
 		)
 	)
-	(label "PCIe_{B1x4}.TX2+"
+	(label "PCIe_B1x4.TX2+"
 		(at 68.58 105.41 0)
 		(effects
@@
 		)
 	)
-	(label "PCIe_{B1x4}.TX3-"
+	(label "PCIe_B1x4.TX3-"
 		(at 68.58 123.19 0)
 		(effects
@@
 		)
 	)
-	(label "PCIe_{B1x4}.RX3-"
+	(label "PCIe_B1x4.RX3-"
 		(at 68.58 130.81 0)
 		(effects
@@
 		)
 	)
-	(label "PCIe_{B1x4}.RX2+"
+	(label "PCIe_B1x4.RX2+"
 		(at 68.58 113.03 0)
 		(effects
@@
 		)
 	)
-	(label "PCIe_{B1x4}.RX0+"
+	(label "PCIe_B1x4.RX0+"
 		(at 68.58 82.55 0)
 		(effects
@@
 		)
 	)
-	(label "PCIE_{REF0}.CK+"
+	(label "PCIE_REF0.CK+"
 		(at 110.49 66.04 180)
 		(effects
@@
 		)
 	)
-	(label "PCIe_{B1x4}.TX1+"
+	(label "PCIe_B1x4.TX1+"
 		(at 68.58 90.17 0)
 		(effects
@@
 		)
 	)
-	(label "PCIe_{B1x4}.TX3+"
+	(label "PCIe_B1x4.TX3+"
 		(at 68.58 120.65 0)
 		(effects
@@
 		)
 	)
-	(label "PCIe_{B1x4}.TX2-"
+	(label "PCIe_B1x4.TX2-"
 		(at 68.58 107.95 0)
 		(effects
@@
 		)
 	)
-	(label "PCIe_{B1x4}.TX0-"
+	(label "PCIe_B1x4.TX0-"
 		(at 68.58 77.47 0)
 		(effects
@@
 		)
 	)
-	(label "PCIe_{B1x4}.RX3+"
+	(label "PCIe_B1x4.RX3+"
 		(at 68.58 128.27 0)
 		(effects
@@
 		)
 	)
-	(label "PCIe_{B1x4}.RX0-"
+	(label "PCIe_B1x4.RX0-"
 		(at 68.58 85.09 0)
 		(effects
@@
 		)
 	)
-	(label "PCIe_{B1x4}.TX1-"
+	(label "PCIe_B1x4.TX1-"
 		(at 68.58 92.71 0)
 		(effects
@@
 		)
 	)
-	(label "PCIE_{REF0}.CK-"
+	(label "PCIE_REF0.CK-"
 		(at 110.49 68.58 180)
 		(effects
@@
 		)
 	)
-	(label "PCIe_{B1x4}.RX2-"
+	(label "PCIe_B1x4.RX2-"
 		(at 68.58 115.57 0)
 		(effects
@@
 		)
 	)
-	(label "PCIe_{B1x4}.TX0+"
+	(label "PCIe_B1x4.TX0+"
 		(at 68.58 74.93 0)
 		(effects
@@
 		)
 	)
-	(label "PCIe_{B1x4}.RX1+"
+	(label "PCIe_B1x4.RX1+"
 		(at 68.58 97.79 0)
 		(effects
@@
 		)
 	)
-	(label "PCIe_{B1x4}.RX1-"
+	(label "PCIe_B1x4.RX1-"
 		(at 68.58 100.33 0)
 		(effects
@@
 		)
 	)
-	(hierarchical_label "PCIE_{REF0}{PCIe_{REF}}"
+	(hierarchical_label "PCIE_REF0{PCIe_REF}"
 		(shape input)
 		(at 59.69 60.96 180)
@@
 		)
 	)
-	(hierarchical_label "PCIe_{B1x4}{PCIe}"
+	(hierarchical_label "PCIe_B1x4{PCIe}"
 		(shape input)
 		(at 59.69 68.58 180)
