File: PC_ExtensionBoard/PC_Coreboard.kicad_sch (KiCad schematic)
At the start: 9 parts, among them U3 KBLH-E61_COMe_Type6_16U

Commit message: update schematic
Connections:
- net LID: now reaches U3.A103 (LID#)
- net PWM: now reaches U3.B101 (FAN_PWMOUT)
- net TACH: now reaches U3.B102 (FAN_TACHIN)
- net SMB_CK: now reaches U3.B13 (SMB_CK)
- net SMB_DAT: now reaches U3.B14 (SMB_DAT)
- net SMB_ALERT: now reaches U3.B15 (SMB_ALERT#)
- net SMB_I2C_CK: now reaches U3.B33 (I2C_CK)
- net SMB_I2C_DAT: now reaches U3.B34 (I2C_DAT)
- net ~{GBE0_LINK_1000}: no longer names the net of U3.A5 (GBE0_LINK1000#)
- now unconnected: U3.B84 (VCC_5V_SBY), U3.B85 (VCC_5V_SBY), U3.B86 (VCC_5V_SBY), U3.B87 (VCC_5V_SBY)
- no-connect marks 3 -> 160

Commit message: update LCSC Number
Connections:
- net DDI1.SCL: no longer U3.C32 (DDI2_CTRLCLK_AUX+)
- net DDI1.SDA: no longer U3.C33 (DDI2_CTRLDATA_AUX-)
- net DDI1.TX0+: no longer U3.D39 (DDI2_PAIR0+)
- net DDI1.TX0-: no longer U3.D40 (DDI2_PAIR0-)
- net DDI1.TX1+: no longer U3.D42 (DDI2_PAIR1+)
- net DDI1.TX1-: no longer U3.D43 (DDI2_PAIR1-)
- net DDI1.TX2+: no longer U3.D46 (DDI2_PAIR2+)
- net DDI1.TX2-: no longer U3.D47 (DDI2_PAIR2-)
- net DDI1.TX3+: no longer U3.D49 (DDI2_PAIR3+)
- net DDI1.TX3-: no longer U3.D50 (DDI2_PAIR3-)
- net DDI1_HPD: no longer U3.D44 (DDI2_HPD)
- net BITCLK renamed HDA.BITCLK
- net PWM renamed FAN.PWM
- net RST renamed HDA.RST
- net SDIN0 renamed HDA.SDIN0
- net SDOUT renamed HDA.SDOUT
- net SPKR renamed HDA.SPKR
- net SYNC renamed HDA.SYNC
- net TACH renamed FAN.TACH
- new net DDI2.SCL: U3.C32 (DDI2_CTRLCLK_AUX+)
- new net DDI2.SDA: U3.C33 (DDI2_CTRLDATA_AUX-)
- new net DDI2.TX0+: U3.D39 (DDI2_PAIR0+)
- new net DDI2.TX0-: U3.D40 (DDI2_PAIR0-)
- new net DDI2.TX1+: U3.D42 (DDI2_PAIR1+)
- new net DDI2.TX1-: U3.D43 (DDI2_PAIR1-)
- new net DDI2.TX2+: U3.D46 (DDI2_PAIR2+)
- new net DDI2.TX2-: U3.D47 (DDI2_PAIR2-)
- new net DDI2.TX3+: U3.D49 (DDI2_PAIR3+)
- new net DDI2.TX3-: U3.D50 (DDI2_PAIR3-)
- new net DDI2_HPD: U3.D44 (DDI2_HPD)
- no-connect marks 160 -> 184

Commit message: update Schematic
Connections:
- net PWR_OK: now reaches U3.B24 (PWR_OK)
- net SATA0-1_SATA_PCIE: now reaches U3.B99 (SATA0-1_SATA_PCIE)
- net PCIE1-4_SATA_PCIE: now reaches U3.B98 (PCIE1-4_SATA_PCIE)
- no-connect marks 184 -> 182
Changed lines of the file:
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@@
 	)
 	(no_connect
+		(at 265.43 328.93)
+	)
+	(no_connect
 		(at 421.64 256.54)
 	)
@@
 	)
 	(no_connect
-		(at 67.31 105.41)
-	)
-	(no_connect
 		(at 214.63 139.7)
 	)
@@
 	)
 	(no_connect
-		(at 265.43 321.31)
-	)
-	(no_connect
 		(at 472.44 143.51)
 	)
@@
 	)
 	(no_connect
-		(at 265.43 250.19)
-	)
-	(no_connect
 		(at 472.44 292.1)
 	)
@@
 	(wire
 		(pts
+			(xy 265.43 250.19) (xy 270.51 250.19)
+		)
+		(stroke
+			(width 0)
+			(type default)
+		)
+	)
+	(wire
+		(pts
 			(xy 118.11 153.67) (xy 118.11 156.21)
 		)
@@
 	(wire
 		(pts
+			(xy 265.43 321.31) (xy 267.97 321.31)
+		)
+		(stroke
+			(width 0)
+			(type default)
+		)
+	)
+	(wire
+		(pts
 			(xy 118.11 77.47) (xy 118.11 80.01)
 		)
@@
 	(wire
 		(pts
+			(xy 63.5 105.41) (xy 67.31 105.41)
+		)
+		(stroke
+			(width 0)
+			(type default)
+		)
+	)
+	(wire
+		(pts
 			(xy 118.11 148.59) (xy 118.11 151.13)
 		)
@@
 		)
 	)
+	(hierarchical_label "SATA0-1_SATA_PCIE"
+		(shape input)
+		(at 270.51 250.19 0)
+		(effects
+			(font
+				(size 1.27 1.27)
+			)
+			(justify left)
+		)
+	)
 	(hierarchical_label "USB3{USB}"
 		(shape output)
@@
 		)
 	)
+	(hierarchical_label "PWR_OK"
+		(shape input)
+		(at 63.5 105.41 180)
+		(effects
+			(font
+				(size 1.27 1.27)
+			)
+			(justify right)
+		)
+	)
 	(hierarchical_label "DDI1{DDI}"
 		(shape input)
@@
 		)
 	)
+	(hierarchical_label "PCIE1-4_SATA_PCIE"
+		(shape input)
+		(at 267.97 321.31 0)
+		(effects
+			(font
+				(size 1.27 1.27)
+			)
+			(justify left)
+		)
+	)

Commit message: bug fixes
Parts:
- U3: footprint DatCao_FootPrint:CORE_BOARD_CUSTOM_440_PIN -> PC_Components_1:EPT_401-51501-51
Connections:
- net PCIE_{REF}.CK+ renamed PCIE_REF.CK+
- net PCIE_{REF}.CK- renamed PCIE_REF.CK-
- net PCIe_{B1x2}.RX0+ renamed PCIe_B1x2.RX0+
- net PCIe_{B1x2}.RX0- renamed PCIe_B1x2.RX0-
- net PCIe_{B1x2}.RX1+ renamed PCIe_B1x2.RX1+
- net PCIe_{B1x2}.RX1- renamed PCIe_B1x2.RX1-
- net PCIe_{B1x2}.TX0+ renamed PCIe_B1x2.TX0+
- net PCIe_{B1x2}.TX0- renamed PCIe_B1x2.TX0-
- net PCIe_{B1x2}.TX1+ renamed PCIe_B1x2.TX1+
- net PCIe_{B1x2}.TX1- renamed PCIe_B1x2.TX1-
- net PCIe_{B1x4}.RX0+ renamed PCIe_B1x4.RX0+
- net PCIe_{B1x4}.RX0- renamed PCIe_B1x4.RX0-
- net PCIe_{B1x4}.RX1+ renamed PCIe_B1x4.RX1+
- net PCIe_{B1x4}.RX1- renamed PCIe_B1x4.RX1-
- net PCIe_{B1x4}.RX2+ renamed PCIe_B1x4.RX2+
- net PCIe_{B1x4}.RX2- renamed PCIe_B1x4.RX2-
- net PCIe_{B1x4}.RX3+ renamed PCIe_B1x4.RX3+
- net PCIe_{B1x4}.RX3- renamed PCIe_B1x4.RX3-
- net PCIe_{B1x4}.TX0+ renamed PCIe_B1x4.TX0+
- net PCIe_{B1x4}.TX0- renamed PCIe_B1x4.TX0-
- net PCIe_{B1x4}.TX1+ renamed PCIe_B1x4.TX1+
- net PCIe_{B1x4}.TX1- renamed PCIe_B1x4.TX1-
- net PCIe_{B1x4}.TX2+ renamed PCIe_B1x4.TX2+
- net PCIe_{B1x4}.TX2- renamed PCIe_B1x4.TX2-
- net PCIe_{B1x4}.TX3+ renamed PCIe_B1x4.TX3+
- net PCIe_{B1x4}.TX3- renamed PCIe_B1x4.TX3-
- no-connect marks 182 -> 186
Changed lines of the file:
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@@
 	)
 	(no_connect
+		(at 472.44 317.5)
+	)
+	(no_connect
 		(at 265.43 316.23)
 	)
@@
 	)
 	(no_connect
+		(at 472.44 320.04)
+	)
+	(no_connect
 		(at 214.63 139.7)
 	)
@@
 	)
 	(no_connect
+		(at 472.44 314.96)
+	)
+	(no_connect
 		(at 265.43 306.07)
 	)
@@
 	)
 	(no_connect
+		(at 472.44 312.42)
+	)
+	(no_connect
 		(at 421.64 46.99)
 	)
@@
 		)
 	)
+	(bus
+		(pts
+			(xy 26.8224 0.1524) (xy 0.1524 0.1524)
+		)
+		(stroke
+			(width 0)
+			(type default)
+		)
+	)
 	(wire
 		(pts
@@
 		)
 	)
-	(label "PCIe_{B1x2}.TX0+"
+	(label "PCIe_B1x2.TX0+"
 		(at 267.97 285.75 0)
 		(effects
@@
 		)
 	)
-	(label "PCIe_{B1x4}.TX2-"
+	(label "PCIe_B1x4.TX2-"
 		(at 214.63 308.61 180)
 		(effects
@@
 		)
 	)
-	(label "PCIe_{B1x4}.TX3+"
+	(label "PCIe_B1x4.TX3+"
 		(at 214.63 316.23 180)
 		(effects
@@
 		)
 	)
-	(label "PCIe_{B1x2}.RX0+"
+	(label "PCIe_B1x2.RX0+"
 		(at 267.97 280.67 0)
 		(effects
@@
 		)
 	)
-	(label "PCIe_{B1x2}.RX1-"
+	(label "PCIe_B1x2.RX1-"
 		(at 267.97 293.37 0)
 		(effects
@@
 		)
 	)
-	(label "PCIe_{B1x4}.RX1-"
+	(label "PCIe_B1x4.RX1-"
 		(at 214.63 293.37 180)
 		(effects
@@
 		)
 	)
-	(label "PCIe_{B1x2}.TX0-"
+	(label "PCIe_B1x2.TX0-"
 		(at 267.97 288.29 0)
 		(effects
@@
 		)
 	)
-	(label "PCIe_{B1x4}.RX3-"
+	(label "PCIe_B1x4.RX3-"
 		(at 214.63 313.69 180)
 		(effects
@@
 		)
 	)
-	(label "PCIe_{B1x4}.RX0-"
+	(label "PCIe_B1x4.RX0-"
 		(at 214.63 283.21 180)
 		(effects
@@
 		)
 	)
-	(label "PCIe_{B1x4}.TX0+"
+	(label "PCIe_B1x4.TX0+"
 		(at 214.63 285.75 180)
 		(effects
@@
 		)
 	)
-	(label "PCIe_{B1x4}.RX3+"
+	(label "PCIe_B1x4.RX3+"
 		(at 214.63 311.15 180)
 		(effects
@@
 		)
 	)
-	(label "PCIe_{B1x2}.RX1+"
+	(label "PCIe_B1x2.RX1+"
 		(at 267.97 290.83 0)
 		(effects
@@
 		)
 	)
-	(label "PCIe_{B1x2}.TX1+"
+	(label "PCIe_B1x2.TX1+"
 		(at 267.97 295.91 0)
 		(effects
@@
 		)
 	)
-	(label "PCIe_{B1x4}.RX1+"
+	(label "PCIe_B1x4.RX1+"
 		(at 214.63 290.83 180)
 		(effects
@@
 		)
 	)
-	(label "PCIe_{B1x2}.TX1-"
+	(label "PCIe_B1x2.TX1-"
 		(at 267.97 298.45 0)
 		(effects
@@
 		)
 	)
-	(label "PCIe_{B1x4}.RX2-"
+	(label "PCIe_B1x4.RX2-"
 		(at 214.63 303.53 180)
 		(effects
@@
 		)
 	)
-	(label "PCIe_{B1x4}.RX2+"
+	(label "PCIe_B1x4.RX2+"
 		(at 214.63 300.99 180)
 		(effects
@@
 		)
 	)
-	(label "PCIe_{B1x4}.TX3-"
+	(label "PCIe_B1x4.TX3-"
 		(at 214.63 318.77 180)
 		(effects
@@
 		)
 	)
-	(label "PCIe_{B1x4}.TX2+"
+	(label "PCIe_B1x4.TX2+"
 		(at 214.63 306.07 180)
 		(effects
@@
 		)
 	)
-	(label "PCIE_{REF}.CK+"
+	(label "PCIE_REF.CK+"
 		(at 204.47 332.74 180)
 		(effects
@@
 		)
 	)
-	(label "PCIe_{B1x4}.RX0+"
+	(label "PCIe_B1x4.RX0+"
 		(at 214.63 280.67 180)
 		(effects
@@
 		)
 	)
-	(label "PCIe_{B1x4}.TX1+"
+	(label "PCIe_B1x4.TX1+"
 		(at 214.63 295.91 180)
 		(effects
@@
 		)
 	)
-	(label "PCIE_{REF}.CK-"
+	(label "PCIE_REF.CK-"
 		(at 204.47 335.28 180)
 		(effects
@@
 		)
 	)
-	(label "PCIe_{B1x4}.TX1-"
+	(label "PCIe_B1x4.TX1-"
 		(at 214.63 298.45 180)
 		(effects
@@
 		)
 	)
-	(label "PCIe_{B1x2}.RX0-"
+	(label "PCIe_B1x2.RX0-"
 		(at 267.97 283.21 0)
 		(effects
@@
 		)
 	)
-	(label "PCIe_{B1x4}.TX0-"
+	(label "PCIe_B1x4.TX0-"
 		(at 214.63 288.29 180)
 		(effects
@@
 		)
 	)
-	(hierarchical_label "PCIE_{REF}{PCIe_{REF}}"
+	(hierarchical_label "PCIE_REF{PCIe_REF}"
 		(shape output)
 		(at 184.15 328.93 180)
@@
 		)
 	)
-	(hierarchical_label "PCIe_{B1x2}{PCIe}"
+	(hierarchical_label "PCIe_B1x2{PCIe}"
 		(shape output)
 		(at 288.29 300.99 0)
@@
 		)
 	)
-	(hierarchical_label "PCIe_{B1x4}{PCIe}"
+	(hierarchical_label "PCIe_B1x4{PCIe}"
 		(shape output)
 		(at 191.77 322.58 180)
@@
 			)
 		)
-		(property "Footprint" "DatCao_FootPrint:CORE_BOARD_CUSTOM_440_PIN"
+		(property "Footprint" "PC_Components_1:EPT_401-51501-51"
 			(at 82.55 115.57 0)
 			(hide yes)
@@
 			)
 		)
-		(property "Footprint" "DatCao_FootPrint:CORE_BOARD_CUSTOM_440_PIN"
+		(property "Footprint" "PC_Components_1:EPT_401-51501-51"
 			(at 436.88 283.21 0)
 			(hide yes)
@@
 			)
 		)
-		(property "Footprint" "DatCao_FootPrint:CORE_BOARD_CUSTOM_440_PIN"
+		(property "Footprint" "PC_Components_1:EPT_401-51501-51"
 			(at 229.87 194.31 0)
 			(hide yes)
@@
 			)
 		)
-		(property "Footprint" "DatCao_FootPrint:CORE_BOARD_CUSTOM_440_PIN"
+		(property "Footprint" "PC_Components_1:EPT_401-51501-51"
 			(at 436.88 252.73 0)
 			(hide yes)
@@
 			)
 		)
-		(property "Footprint" "DatCao_FootPrint:CORE_BOARD_CUSTOM_440_PIN"
+		(property "Footprint" "PC_Components_1:EPT_401-51501-51"
 			(at 85.09 262.89 0)
 			(hide yes)
@@
 			)
 		)
-		(property "Footprint" "DatCao_FootPrint:CORE_BOARD_CUSTOM_440_PIN"
+		(property "Footprint" "PC_Components_1:EPT_401-51501-51"
 			(at 436.88 71.12 0)
 			(hide yes)
@@
 			)
 		)
-		(property "Footprint" "DatCao_FootPrint:CORE_BOARD_CUSTOM_440_PIN"
+		(property "Footprint" "PC_Components_1:EPT_401-51501-51"
 			(at 436.88 143.51 0)
 			(hide yes)
@@
 			)
 		)
-		(property "Footprint" "DatCao_FootPrint:CORE_BOARD_CUSTOM_440_PIN"
+		(property "Footprint" "PC_Components_1:EPT_401-51501-51"
 			(at 229.87 236.22 0)
 			(hide yes)
@@
 			)
 		)
-		(property "Footprint" "DatCao_FootPrint:CORE_BOARD_CUSTOM_440_PIN"
+		(property "Footprint" "PC_Components_1:EPT_401-51501-51"
 			(at 229.87 303.53 0)
 			(hide yes)
@@
 			)
 		)
-		(property "Footprint" "DatCao_FootPrint:CORE_BOARD_CUSTOM_440_PIN"
+		(property "Footprint" "PC_Components_1:EPT_401-51501-51"
 			(at 436.88 187.96 0)
 			(hide yes)
@@
 			)
 		)
-		(property "Footprint" "DatCao_FootPrint:CORE_BOARD_CUSTOM_440_PIN"
+		(property "Footprint" "PC_Components_1:EPT_401-51501-51"
 			(at 436.88 320.04 0)
 			(hide yes)
@@
 			)
 		)
-		(property "Footprint" "DatCao_FootPrint:CORE_BOARD_CUSTOM_440_PIN"
+		(property "Footprint" "PC_Components_1:EPT_401-51501-51"
 			(at 229.87 129.54 0)
 			(hide yes)
@@
 			)
 		)
-		(property "Footprint" "DatCao_FootPrint:CORE_BOARD_CUSTOM_440_PIN"
+		(property "Footprint" "PC_Components_1:EPT_401-51501-51"
 			(at 85.09 346.71 0)
 			(hide yes)
@@
 			)
 		)
-		(property "Footprint" "DatCao_FootPrint:CORE_BOARD_CUSTOM_440_PIN"
+		(property "Footprint" "PC_Components_1:EPT_401-51501-51"
 			(at 436.88 219.71 0)
 			(hide yes)
@@
 			)
 		)
-		(property "Footprint" "DatCao_FootPrint:CORE_BOARD_CUSTOM_440_PIN"
+		(property "Footprint" "PC_Components_1:EPT_401-51501-51"
 			(at 229.87 62.23 0)
 			(hide yes)
@@
 			)
 		)
-		(property "Footprint" "DatCao_FootPrint:CORE_BOARD_CUSTOM_440_PIN"
+		(property "Footprint" "PC_Components_1:EPT_401-51501-51"
 			(at 85.09 304.8 0)
 			(hide yes)
