File: PC_ExtensionBoard/PC_ExtensionBoard.kicad_sch (KiCad schematic)
At the start: 0 parts

Commit message: bug fixes
Other:
- sheet M.2 Key E ports: added PCIE_REF3{PCIe_REF}, PCIe_B1x2{PCIe}; removed PCIE_{REF3}{PCIe_{REF}}, PCIe_{B1x2}{PCIe}
- sheet M.2 Key M #1 ports: added PCIE_REF0{PCIe_REF}, PCIe_B1x4{PCIe}; removed PCIE_{REF0}{PCIe_{REF}}, PCIe_{B1x4}{PCIe}
- sheet MISC ports: added PCIE_REF0{PCIe_REF}, PCIE_REF3{PCIe_REF}, PCIE_REFIN{PCIe_REF}; removed PCIE_{REF0}{PCIe_{REF}}, PCIE_{REF3}{PCIe_{REF}}, PCIE_{REFIN}{PCIe_{REF}}
- sheet PC_CoreBoard ports: added PCIE_REF{PCIe_REF}, PCIe_B1x2{PCIe}, PCIe_B1x4{PCIe}; removed PCIE_{REF}{PCIe_{REF}}, PCIe_{B1x2}{PCIe}, PCIe_{B1x4}{PCIe}
Changed lines of the file:
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@@
+	)
+	(no_connect
+		(at 204.47 260.35)
 	)
 	(no_connect
@@
 	)
 	(no_connect
-		(at 266.7 241.3)
-	)
-	(no_connect
 		(at 251.46 241.3)
 	)
@@
 	)
 	(no_connect
+		(at 204.47 257.81)
+	)
+	(no_connect
 		(at 350.52 180.34)
 	)
@@
 	)
 	(no_connect
-		(at 259.08 241.3)
-	)
-	(no_connect
 		(at 368.3 180.34)
 	)
@@
 	(bus
 		(pts
-			(xy 312.42 261.62) (xy 326.39 261.62)
+			(xy 312.42 265.43) (xy 326.39 265.43)
 		)
 		(stroke
@@
 		)
 	)
-	(bus
-		(pts
-			(xy 312.42 265.43) (xy 340.36 265.43)
-		)
-		(stroke
-			(width 0)
-			(type default)
-		)
-	)
 	(wire
 		(pts
@@
 	(bus
 		(pts
-			(xy 326.39 261.62) (xy 326.39 237.49)
+			(xy 326.39 265.43) (xy 326.39 237.49)
 		)
 		(stroke
@@
 		(pts
 			(xy 195.58 247.65) (xy 204.47 247.65)
+		)
+		(stroke
+			(width 0)
+			(type default)
+		)
+	)
+	(bus
+		(pts
+			(xy 312.42 273.05) (xy 340.36 273.05)
 		)
 		(stroke
@@
 			)
 		)
-		(pin "PCIe_{B1x2}{PCIe}" output
-			(at 248.92 322.58 270)
-			(effects
-				(font
-					(size 1.27 1.27)
-				)
-				(justify left)
-			)
-		)
-		(pin "PCIe_{B1x4}{PCIe}" output
-			(at 312.42 265.43 0)
-			(effects
-				(font
-					(size 1.27 1.27)
-				)
-				(justify right)
-			)
-		)
 		(pin "USB_0_1_OC#" output
 			(at 204.47 267.97 180)
@@
 			)
 		)
-		(pin "PCIE_{REF}{PCIe_{REF}}" output
-			(at 309.88 241.3 90)
-			(effects
-				(font
-					(size 1.27 1.27)
-				)
-				(justify right)
-			)
-		)
 		(pin "USB4{USB}" output
-			(at 259.08 241.3 90)
-			(effects
-				(font
-					(size 1.27 1.27)
-				)
-				(justify right)
+			(at 204.47 257.81 180)
+			(effects
+				(font
+					(size 1.27 1.27)
+				)
+				(justify left)
 			)
 		)
@@
 		)
 		(pin "USB6{USB}" output
-			(at 266.7 241.3 90)
-			(effects
-				(font
-					(size 1.27 1.27)
-				)
-				(justify right)
+			(at 204.47 260.35 180)
+			(effects
+				(font
+					(size 1.27 1.27)
+				)
+				(justify left)
 			)
 		)
@@
 		)
 		(pin "SATA0{SATA}" output
-			(at 312.42 261.62 0)
+			(at 312.42 265.43 0)
 			(effects
 				(font
@@
 		(pin "SATA0-1_SATA_PCIE" input
 			(at 295.91 241.3 90)
+			(effects
+				(font
+					(size 1.27 1.27)
+				)
+				(justify right)
+			)
+		)
+		(pin "PCIe_B1x2{PCIe}" output
+			(at 248.92 322.58 270)
+			(effects
+				(font
+					(size 1.27 1.27)
+				)
+				(justify left)
+			)
+		)
+		(pin "PCIe_B1x4{PCIe}" output
+			(at 312.42 273.05 0)
+			(effects
+				(font
+					(size 1.27 1.27)
+				)
+				(justify right)
+			)
+		)
+		(pin "PCIE_REF{PCIe_REF}" output
+			(at 309.88 241.3 90)
 			(effects
 				(font
@@
 			)
 		)
-		(pin "PCIE_{REF0}{PCIe_{REF}}" output
-			(at 438.15 217.17 0)
-			(effects
-				(font
-					(size 1.27 1.27)
-				)
-				(justify right)
-			)
-		)
-		(pin "PCIE_{REFIN}{PCIe_{REF}}" input
-			(at 341.63 224.79 180)
-			(effects
-				(font
-					(size 1.27 1.27)
-				)
-				(justify left)
-			)
-		)
 		(pin "GPIOEX0" output
 			(at 350.52 180.34 90)
@@
 			)
 		)
-		(pin "PCIE_{REF3}{PCIe_{REF}}" output
-			(at 438.15 210.82 0)
-			(effects
-				(font
-					(size 1.27 1.27)
-				)
-				(justify right)
-			)
-		)
 		(pin "SATA0{SATA}" output
 			(at 372.11 228.6 270)
@@
 		(pin "SATA0-1_SATA_PCIE" input
 			(at 341.63 217.17 180)
+			(effects
+				(font
+					(size 1.27 1.27)
+				)
+				(justify left)
+			)
+		)
+		(pin "PCIE_REF3{PCIe_REF}" output
+			(at 438.15 210.82 0)
+			(effects
+				(font
+					(size 1.27 1.27)
+				)
+				(justify right)
+			)
+		)
+		(pin "PCIE_REF0{PCIe_REF}" output
+			(at 438.15 217.17 0)
+			(effects
+				(font
+					(size 1.27 1.27)
+				)
+				(justify right)
+			)
+		)
+		(pin "PCIE_REFIN{PCIe_REF}" input
+			(at 341.63 224.79 180)
 			(effects
 				(font
@@
 			)
 		)
-		(pin "PCIe_{B1x2}{PCIe}" input
+		(pin "PCIE_REF3{PCIe_REF}" input
+			(at 306.07 349.25 0)
+			(effects
+				(font
+					(size 1.27 1.27)
+				)
+				(justify right)
+			)
+		)
+		(pin "PCIe_B1x2{PCIe}" input
 			(at 248.92 334.01 90)
-			(effects
-				(font
-					(size 1.27 1.27)
-				)
-				(justify right)
-			)
-		)
-		(pin "PCIE_{REF3}{PCIe_{REF}}" input
-			(at 306.07 349.25 0)
 			(effects
 				(font
@@
 			)
 		)
-		(pin "PCIe_{B1x4}{PCIe}" input
-			(at 340.36 265.43 180)
-			(effects
-				(font
-					(size 1.27 1.27)
-				)
-				(justify left)
-			)
-		)
-		(pin "PCIE_{REF0}{PCIe_{REF}}" input
+		(pin "PCIe_B1x4{PCIe}" input
+			(at 340.36 273.05 180)
+			(effects
+				(font
+					(size 1.27 1.27)
+				)
+				(justify left)
+			)
+		)
+		(pin "PCIE_REF0{PCIe_REF}" input
 			(at 439.42 260.35 0)
 			(effects
