File: PC_ExtensionBoard/PC_ExtensionBoard.kicad_sch (KiCad schematic)
At the start: 0 parts

Commit message: update
Other:
- removed sheet HDMI
- removed sheet M.2 Key E
- removed sheet M.2 Key M #1
- removed sheet MISC
- removed sheet PC_CoreBoard
- removed sheet Power
- removed sheet USB_RJ45
- added sheet 1_Module_Clock (1_Module_Clock.kicad_sch)
- added sheet 2_Power (2_Power.kicad_sch)
- added sheet 3_PCIe_LAN (3_PCIe_LAN.kicad_sch)
- added sheet 4_USB_SATA (4_USB_SATA.kicad_sch)
- added sheet 5_Display (5_Display.kicad_sch)
- added sheet 6_Audio (6_Audio.kicad_sch)
- added sheet 7_Serial_SuperIO (7_Serial_SuperIO.kicad_sch)
- added sheet 8_Misc_IO (8_Misc_IO.kicad_sch)
